File: bldc_foc_controller/bldc_foc_controller.sch (KiCad schematic (older format))
At the start: 0 parts

Commit message: schem and code
Parts:
- added C?: C_47uF, footprints:C_0805_OEM, symbol formula:C_47uF
- added C? (x3): C_1uF, footprints:C_0805_OEM, symbol formula:C_1uF
- added J? (x2): Conn_02x19_Odd_Even, symbol Connector_Generic:Conn_02x19_Odd_Even
- added J?: CONN_01X03, Pin_Headers:Pin_Header_Straight_1x03_Pitch2.54mm, symbol formula:CONN_01X03
- added J? (x3): CONN_01x02, footprints:PinHeader_1x02_P2.54mm_Vertical, symbol formula:CONN_01x02
- added U?: DRV8350FSRTVR, symbol formula:DRV8350FSRTVR
- added U? (x4): redcube-7461057, formula:redcube_pressfit_6pin, symbol formula:redcube-7461057
Connections:
- net labels added: ANA_MISC0, ANA_MISC_1, CS, DRV_EN, DRV_nFAULT, GHA, GHB, GHC, GLA, GLB, GLC, GND, IN+, IN-, INHA, INHB, INHC, INLA, INLB, INLC, MISO, MOSI, OUT+, OUT-, SCLK, SDI, SDO, SNSHA, SNSHB, SNSHC, SNSLA, SNSLB, SNSLC, THERM_0, THERM_1, UART_RX, UART_TX, VDRAIN
- wire segments 0 -> 20
Other:
- note added: "3 Phase Half Bridge Inverter"
- note added: "47nF x7r"
- note added: "Hall Effect Sensor Input \nFor 6 Step commutation \nw/ jumpers\n(pg 23)"
- note added: "Header plugins for STM32G431 Nucleo board\nNucleo sits underneath motor drive PCB"
- note added: "Interface to uC"
- note added: "Left Side conn"
- note added: "Right Side conn"
- note added: "TI Gate Driver IC"
- note added: "\nhttps://www.st.com/content/ccc/resource/technical/layouts_and_diagrams/schematic_pack/group1/98/d2/70/60/b1/cb/44/4c/mb1367-g431rb-c04_schematic/files/mb1367-g431rb-c04_schematic.pdf/jcr:content/translations/en.mb1367-g431rb-c04_schematic.pdf"

Commit message: schematic updates
Parts:
- added C? (x2): C_.22uF, footprints:C_0805_OEM, symbol formula:C_.22uF
- added C?: C, symbol Device:C
- added C?: C_10pF, footprints:C_0805_OEM, symbol Device:C
- added C?: C_100uF+, footprints:C_100uF+, symbol formula:C_100uF+
- added C?: C_35nF, footprints:C_0805_OEM, symbol Device:C
- added C? (x16): C_10uF, footprints:C_1206_OEM, symbol Device:C
- added C? (x4): C_100uF, Capacitor_THT:CP_Radial_D6.3mm_P2.50mm, symbol Device:CP1
- added C? (x2): C_820uF, Capacitor_THT:CP_Radial_D8.0mm_P3.80mm, symbol Device:CP1
- added D?: D_TVS _39V_ 824551241, footprints:DO-214AB, symbol Device:D_TVS
- added J?: Conn_01x05, symbol Connector_Generic:Conn_01x05
- added L?: SRP0520-4R7K, symbol formula:SRP0520-4R7K
- added Q? (x6): PSMN2R2-40YSD, footprints:LFPAK56, symbol Device:Q_NMOS_SGD
- added Q? (x2): HYG025N06LS1C2, footprints:PDFN_5X6MC_MCH, symbol Device:Q_NMOS_DGS
- added R?: R_120K, footprints:R_0805_OEM, symbol formula:R_120K
- added R?: R, symbol Device:R
- added R? (x2): R_2M, footprints:R_0805_OEM, symbol Device:R
- added R? (x2): R_100K, footprints:R_0805_OEM, symbol formula:R_100K
- added R?: R_22K, footprints:R_0805_OEM, symbol formula:R_22K
- added R? (x4): R_10K, footprints:R_0805_OEM, symbol formula:R_10K
- added R? (x5): R_1m_5W, footprints:HCS3920FT1L00, symbol formula:R_1m_5W
- added R?: R_845K, footprints:R_0805_OEM, symbol Device:R
- added R?: R_1K, footprints:R_0805_OEM, symbol formula:R_1K
- added TP? (x6): Test_Point_SMD, footprints:Test_Point_SMD, symbol formula:Test_Point_SMD
- added U?: TLS4120D0EPVXUMA1, footprints:TLS4120D0EPVXUMA1, symbol formula:TLS4120D0EPVXUMA1
- added U? (x3): INA240A1D, Package_SO:SOIC-8_3.9x4.9mm_P1.27mm, symbol Amplifier_Current:INA240A1D
- added U?: LTC4368CMS-2-PBF, footprints:LTC4368CMS-2-PBF, symbol formula:LTC4368CMS-2-PBF
Connections:
- net labels added: +10V, +3V3, +5V, BUCK_RST, ENCODER_A, ENCODER_B, ENCODER_X, LTC_FAULT, PH_A, PH_C, SNS_HA, SNS_HB, SNS_HC, SNS_LA, SNS_LB, SNS_LC, SNS_SH_A, SNS_SH_B, SNS_SH_C, STM_VREF, THERM_2, USART1_RX, USART1_TX, VBUS_20V, VBUS_SNS_+, VBUS_UNPROTECTED
- net labels removed: ANA_MISC0, ANA_MISC_1, IN+, IN-, SNSHA, SNSHB, SNSHC, SNSLA, SNSLB, SNSLC, UART_RX, UART_TX, VDRAIN
- wire segments 20 -> 231
Other:
- note added: "1206 MLCC X5R Cap Bank\n10uF @50V \nDerates to 1.8uF @25V"
- note added: "20x THT 6.3mm 35v \n100uF 50mohm ESR \nAluminum Polymers"
- note added: "2x THT 820uF \n35V?? 8mm THTs\nAluminum Electrolytics"
- note added: "3 Phase Inverter"
- note added: "40V Power MOSFETS"
- note added: "6 State Hall Effect\nSensor Input\n"
- note added: "Bidirectional High CMRR \nShunt Amplifiers"
- note added: "Input Cap Bank"
- note added: "Left Side \nconn CN7"
- note added: "On-board Optional\nThermistors"
- note added: "Precharge, OV/UV Protection, \nOvercurrent & Reverse Current \nProtection chip"
- note added: "Regulated Board Power\nvia 2.6MHz 10V out 2A Buck"
- note added: "Right Side \nconn CN10"
- note added: "Rotary Encoder Input\nFor AMT103-V \nhttps://www.digikey.com/en/products\n/detail/cui-devices/AMT103-V/827016"
- note added: "Vin"
- note added: "Vout"
- note added: "add PTC fuse? Buck has\ninternal overcurrent limit"
- note added: "layout note: AGND \nconn to GND using \nbroad PCB trace"
- note removed: "2"
- note removed: "3 Phase Half Bridge Inverter"
- note removed: "Hall Effect Sensor Input \nFor 6 Step commutation \nw/ jumpers\n(pg 23)"
- note removed: "Left Side conn"
- note removed: "Right Side conn"
- moved on the sheet: C?, J?, U?

Commit message: schem changes
Parts:
- removed C?: C_47uF, footprints:C_0805_OEM, symbol formula:C_47uF
- removed C? (x3): C_1uF, footprints:C_0805_OEM, symbol formula:C_1uF
- removed D?: D_TVS _39V_ 824551241, footprints:DO-214AB, symbol Device:D_TVS
- removed Q? (x4): PSMN2R2-40YSD, footprints:LFPAK56, symbol Device:Q_NMOS_SGD
- removed Q? (x2): HYG025N06LS1C2, footprints:PDFN_5X6MC_MCH, symbol Device:Q_NMOS_DGS
- removed R? (x3): R_10K, footprints:R_0805_OEM, symbol formula:R_10K
- removed R? (x5): R_1m_5W, footprints:HCS3920FT1L00, symbol formula:R_1m_5W
- removed R?: R_1K, footprints:R_0805_OEM, symbol formula:R_1K
- removed TP? (x4): Test_Point_SMD, footprints:Test_Point_SMD, symbol formula:Test_Point_SMD
- removed U?: DRV8350FSRTVR, symbol formula:DRV8350FSRTVR
- removed U? (x2): INA240A1D, Package_SO:SOIC-8_3.9x4.9mm_P1.27mm, symbol Amplifier_Current:INA240A1D
- added C? (x7): C_10uF, footprints:C_0805_OEM, symbol formula:C_10uF
- added C? (x12): DNP, footprints:C_0805_OEM, symbol Device:C
- added C?: C_100nF, footprints:C_0603_1608Metric, symbol formula:C_100nF
- added C? (x3): C_0.1uF, footprints:C_0805_OEM, symbol formula:C_0.1uF
- added C? (x6): C_10uF, footprints:C_1206_OEM, symbol Device:C
- added C? (x3): C_1uF, footprints:C_0805_OEM, symbol formula:C_1uF
- added C?: C_47uF, footprints:C_0805_OEM, symbol formula:C_47uF
- added D? (x2): D_TVS_35V, SMC_DIO, symbol formula:D_TVS_35V
- added H?: MountingHole_Pad, symbol Mechanical:MountingHole_Pad
- added J?: Conn_01x10, footprints:PinHeader_1x10_P2.54mm_Vertical, symbol formula:Conn_01x10
- added NT? (x2): Net-Tie_2, symbol Device:Net-Tie_2
- added Q? (x4): HYG025N06LS1C2, footprints:PDFN_5X6MC_MCH, symbol Device:Q_NMOS_DGS
- added Q? (x6): DNP, footprints:LFPAK56, symbol Device:Q_NMOS_SGD
- added Q? (x4): PSMN2R2-40YSD, footprints:LFPAK56, symbol Device:Q_NMOS_SGD
- added R? (x6): R_1, footprints:R_0805_OEM, symbol formula:R_1
- added R? (x15): DNP, footprints:R_0805_OEM, symbol Device:R
- added R? (x3): R_10K, footprints:R_0805_OEM, symbol formula:R_10K
- added R? (x6): R_0, footprints:R_0603_1608Metric, symbol formula:R_0
- added R? (x5): R_1m_3W_1%, WSL2726_VIS, symbol formula:R_1m_3W_1%
- added R?: R_1K, footprints:R_0805_OEM, symbol formula:R_1K
- added R?: R_300K, footprints:R_0805_OEM, symbol formula:R_300K
- added R?: R_97.6K, footprints:R_0805_OEM, symbol Device:R
- added TP? (x4): Test_Point_SMD, footprints:Test_Point_SMD, symbol formula:Test_Point_SMD
- added U? (x2): INA240A1D, Package_SO:SOIC-8_3.9x4.9mm_P1.27mm, symbol Amplifier_Current:INA240A1D
- added U?: DRV8320S, footprints:QFN50P500X500X80-33N, symbol formula:DRV8320S
- added U? (x2): LMP8481ASQDGKRQ1, footprints:LMP8481ASQDGKRQ1, symbol formula:LMP8481ASQDGKRQ1
- U?: value LTC4368CMS-2-PBF -> LTC4368CMS-1-PBF
Connections:
- net labels added: A_UNFILTERED, B_UNFILTERED, LOAD_PWM, PH_A_SH, PH_B, PH_B_SH, PH_C_SH, REGEN_LOAD+, REGEN_LOAD_-, REGEN_LOAD_SH_+, REGEN_LOAD_SH_-, SNS_SH_REGEN_LOAD, SNS_SH_SYSTEM, SYSTEM_SH_+, SYSTEM_SH_-, X_UNFILTERED
- net labels removed: BUCK_RST, OUT+, OUT-, VBUS_SNS_+
- wire segments 231 -> 530
Other:
- note added: "20uF MLCC \nlocal bypass cap"
- note added: "40V Power MOSFETS\nDNP'd in Parallel"
- note added: "DNP 10K Pullups for encoder \nDNP RC Filters on output of encoder"
- note added: "DNP'd RC snubbers\nbetween FET D&S"
- note added: "In-phase current sensing"
- note added: "LTC4368 for Precharge, OV/UV\nProtection, Overcurrent & \nReverse Current Protection"
- note added: "On-board Optional\nThermistors w/ filtering"
- note added: "Rotary Encoder"
- note added: "bidirectional shunt amp \nfor system shunt current \nsense"
- note added: "unidirectional shunt amp \nfor load shunt current \nsense"
- note removed: "40V Power MOSFETS"
- note removed: "On-board Optional\nThermistors"
- note removed: "Precharge, OV/UV Protection, \nOvercurrent & Reverse Current \nProtection chip"
- moved on the sheet: C?, J?, L?, Q?, R?, TP?, U?

Commit message: schem changes fr
Other:
- note added: "4x THT 6.3mm 35v \n100uF 50mohm ESR \nAluminum Polymers"
- note removed: "20x THT 6.3mm 35v \n100uF 50mohm ESR \nAluminum Polymers"
Changed lines of the file:
@@
 	9325 975  9725 975
 Text Notes 8725 875  0    50   ~ 0
-20x THT 6.3mm 35v \n100uF 50mohm ESR \nAluminum Polymers
+4x THT 6.3mm 35v \n100uF 50mohm ESR \nAluminum Polymers
 $Comp
 L Device:CP1 C?

Commit message: more schem changes
Parts:
- removed NT?: Net-Tie_2, symbol Device:Net-Tie_2
- removed R? (x6): DNP, footprints:R_0805_OEM, symbol Device:R
- removed R? (x6): R_0, footprints:R_0603_1608Metric, symbol formula:R_0
- added H? (x2): MotorConnector_Pad, symbol Mechanical:MountingHole_Pad
- added NT?: Net-Tie_2, symbol Device:Net-Tie_2
- added R? (x6): R_0_0205, symbol Device:R
- C? (x2): value C_.22uF -> C_220nF
- C? (x3): value C_0.1uF -> C_100nF
- H?: value MountingHole_Pad -> MotorConnector_Pad
- R?: value R_10K -> R_1K
Connections:
- net A_UNFILTERED: now also R?.2
- net B_UNFILTERED: now also R?.2
- net ENCODER_A: now also R?.1
- net ENCODER_B: now also R?.1
- net ENCODER_X: now also R?.1
- net GND: no longer C?.2, R?.2, R?.2
- net PH_A: now also H?.1
- net PH_B: now also H?.1
- net PH_C: now also H?.1
- net SNS_SH_A: now also R?.1
- net SNS_SH_B: now also R?.1
- net SNS_SH_C: now also R?.1
- net X_UNFILTERED: now also R?.2
- net at R?.1: now also U?.1 (FREQ)
- net at U?.12 (SSON): now also C?.2, R?.2, R?.2, U?.4 (AGND), NT?.2
- net at U?.15 (EPAD): now also NT?.1
- net at U?.5: now also R?.2 (x3)
Other:
- note added: "MOTOR CONNECTORS\n"
- moved on the sheet: R?

Commit message: more schem chagnes
Parts:
- removed C?: C, symbol Device:C
- removed R?: R, symbol Device:R
- removed R? (x5): R_0_0205, symbol Device:R
- removed R?: R_1K, footprints:R_0805_OEM, symbol formula:R_1K
- removed R?: R_1K, footprints:R_0805_OEM, symbol formula:R_10K
- added D? (x3): D_TVS_35V, SMC_DIO, symbol formula:D_TVS_35V
- added R? (x5): R_0, footprints:R_0805_OEM, symbol Device:R
- added R? (x4): R_10K, footprints:R_0805_OEM, symbol formula:R_10K
- R?: value R_0_0205 -> R_0; footprint (none) -> footprints:R_0805_OEM
Connections:
- net +3V3: now also R?.1, R?.1, R?.2, R?.2
- net A_UNFILTERED: now also R?.2
- net B_UNFILTERED: now also R?.2
- net CS: now also R?.1
- net DRV_EN: now also R?.2
- net DRV_nFAULT: now also R?.1
- net ENCODER_A: now also R?.1
- net ENCODER_B: now also R?.1
- net GND: now also NT?.1, U?.15 (EPAD), D?.2, D?.2, D?.2
- net PH_A: now also D?.1
- net PH_B: now also D?.1
- net PH_B_SH: now also C?.2, R?.2
- net PH_C: now also D?.1
- net SDO: now also R?.2
- net SNS_SH_A: now also R?.1
- net SNS_SH_B: now also R?.1
- net SNS_SH_C: now also R?.1
- net at U?.5: now also R?.2 (x3)
Other:
- note added: "Buck Converter\n"
- note added: "Current Sensing"
- note added: "Misc. Headers"
- note added: "Motor phase current sensing"
- note added: "Precharge Circuitry"
- note added: "Quadrature Encoder Inputs"
- note added: "STM32 Nucleo"
- note added: "Unidirectional TVS \ndiodes for ESD protection"
- note removed: "In-phase current sensing"
- note removed: "Rotary Encoder"
- moved on the sheet: C?, H?, J?, L?, NT?, Q?, R?, TP?, U?

Commit message: simple changes yuh
Parts:
- added R?: R_1.54K, footprints:R_0805_OEM, symbol formula:R_1.54K
- added U?: R_500, footprints:R_0805_OEM, symbol formula:R_500
Connections:
- net GND: now also U?.2
- net VBUS_UNPROTECTED: now also R?.1
- new net SHDN: R?.2, U?.1
Other:
- moved on the sheet: D?, R?
Changed lines of the file:
@@
 	1    0    0    -1
 $EndComp
-Connection ~ 3950 3500
 $Comp
 L power:+10V #PWR0109
@@
 L Device:R R?
 U 1 1 61B4CA23
-P 2850 2450
-F 0 "R?" H 2920 2496 50  0000 L CNN
-F 1 "R_845K" H 2925 2400 50  0000 L CNN
-F 2 "footprints:R_0805_OEM" V 2780 2450 50  0001 C CNN
-F 3 "https://www.digikey.com/en/products/detail/stackpole-electronics-inc/RMCF0805FT845K/1713403" H 2850 2450 50  0001 C CNN
-	1    2850 2450
+P 2600 2450
+F 0 "R?" H 2670 2496 50  0000 L CNN
+F 1 "R_845K" H 2675 2400 50  0000 L CNN
+F 2 "footprints:R_0805_OEM" V 2530 2450 50  0001 C CNN
+F 3 "https://www.digikey.com/en/products/detail/stackpole-electronics-inc/RMCF0805FT845K/1713403" H 2600 2450 50  0001 C CNN
+	1    2600 2450
 	1    0    0    -1
 $EndComp
@@
 L Device:R R?
 U 1 1 61B5D3A0
-P 2850 2750
-F 0 "R?" H 2920 2796 50  0000 L CNN
-F 1 "R_2M" H 2920 2705 50  0000 L CNN
-F 2 "footprints:R_0805_OEM" V 2780 2750 50  0001 C CNN
-F 3 "https://www.digikey.com/en/products/detail/stackpole-electronics-inc/RMCF0805FT2M00/1760219" H 2850 2750 50  0001 C CNN
-	1    2850 2750
+P 2600 2750
+F 0 "R?" H 2670 2796 50  0000 L CNN
+F 1 "R_2M" H 2670 2705 50  0000 L CNN
+F 2 "footprints:R_0805_OEM" V 2530 2750 50  0001 C CNN
+F 3 "https://www.digikey.com/en/products/detail/stackpole-electronics-inc/RMCF0805FT2M00/1760219" H 2600 2750 50  0001 C CNN
+	1    2600 2750
 	1    0    0    -1
 $EndComp
@@
 Connection ~ 1075 3500
 Wire Wire Line
-	1075 3500 1900 3500
+	1075 3500 1825 3500
 Text Label 1100 3500 0    50   ~ 0
 REGEN_LOAD_-
@@
 Text Label 4225 10050 0    50   ~ 0
 SNS_SH_SYSTEM
-Connection ~ 2850 1425
-Wire Wire Line
-	2850 1425 3025 1425
 $Comp
 L formula:R_300K R?
 U 1 1 692D0260
-P 2850 3050
-F 0 "R?" H 2920 3096 50  0000 L CNN
-F 1 "R_300K" H 2920 3005 50  0000 L CNN
-F 2 "footprints:R_0805_OEM" H 2780 3050 50  0001 C CNN
-F 3 "https://industrial.panasonic.com/cdbs/www-data/pdf/RDM0000/AOA0000C307.pdf" H 2930 3050 50  0001 C CNN
-F 4 "DK" H 2850 3050 60  0001 C CNN "MFN"
-F 5 "P300KDACT-ND" H 2850 3050 60  0001 C CNN "MPN"
-F 6 "https://www.digikey.com/product-detail/en/panasonic-electronic-components/ERA-6AEB304V/P300KDACT-ND/1466006" H 3330 3450 60  0001 C CNN "PurchasingLink"
-	1    2850 3050
+P 2600 3050
+F 0 "R?" H 2670 3096 50  0000 L CNN
+F 1 "R_300K" H 2670 3005 50  0000 L CNN
+F 2 "footprints:R_0805_OEM" H 2530 3050 50  0001 C CNN
+F 3 "https://industrial.panasonic.com/cdbs/www-data/pdf/RDM0000/AOA0000C307.pdf" H 2680 3050 50  0001 C CNN
+F 4 "DK" H 2600 3050 60  0001 C CNN "MFN"
+F 5 "P300KDACT-ND" H 2600 3050 60  0001 C CNN "MPN"
+F 6 "https://www.digikey.com/product-detail/en/panasonic-electronic-components/ERA-6AEB304V/P300KDACT-ND/1466006" H 3080 3450 60  0001 C CNN "PurchasingLink"
+	1    2600 3050
 	1    0    0    -1
 $EndComp
@@
 L Device:R R?
 U 1 1 693C1FA4
-P 2850 3350
-F 0 "R?" H 2920 3396 50  0000 L CNN
-F 1 "R_97.6K" H 2920 3305 50  0000 L CNN
-F 2 "footprints:R_0805_OEM" V 2780 3350 50  0001 C CNN
-F 3 "~" H 2850 3350 50  0001 C CNN
-	1    2850 3350
+P 2600 3350
+F 0 "R?" H 2670 3396 50  0000 L CNN
+F 1 "R_97.6K" H 2670 3305 50  0000 L CNN
+F 2 "footprints:R_0805_OEM" V 2530 3350 50  0001 C CNN
+F 3 "~" H 2600 3350 50  0001 C CNN
+	1    2600 3350
 	1    0    0    -1
 $EndComp
-Connection ~ 2850 3500
+Connection ~ 2600 3500
 Wire Wire Line
 	3525 3100 3525 3200
 Wire Wire Line
-	3250 2200 2850 2200
-Wire Wire Line
-	2850 1425 2850 2200
-Connection ~ 2850 2200
+	2600 1425 2600 2200
+Connection ~ 2600 2200
 Wire Wire Line
 	3550 2200 3600 2200
@@
 $Comp
 L formula:D_TVS_35V D?
-U 1 1 61F5EEBD
-P 2375 2600
-F 0 "D?" H 2625 2475 60  0000 R CNN
-F 1 "D_TVS_35V" H 2800 2725 60  0000 R CNN
-F 2 "SMC_DIO" H 2575 2240 60  0001 C CNN
-F 3 "https://www.diodes.com/assets/Datasheets/ds40741.pdf" H 2375 2600 60  0001 C CNN
-F 4 "SMCJ22A-13-F" H 2525 2850 50  0001 C CNN "MPN"
-	1    2375 2600
-	0    -1   -1   0
-$EndComp
-$Comp
-L formula:D_TVS_35V D?
 U 1 1 61FF9FF0
 P 5850 2450
@@
 	0    -1   -1   0
 $EndComp
-Wire Wire Line
-	2375 2600 2375 3500
-Wire Wire Line
-	2375 3500 2850 3500
-Wire Wire Line
-	2375 2200 2375 1425
-Wire Wire Line
-	1075 1425 2375 1425
-Connection ~ 2375 1425
-Wire Wire Line
-	2375 1425 2850 1425
 $Comp
 L Mechanical:MountingHole_Pad H?
@@
 Wire Wire Line
 	9250 7700 9425 7700
-Connection ~ 2850 2900
-Connection ~ 2850 3200
-Wire Wire Line
-	2850 2900 3425 2900
-Wire Wire Line
-	2850 3200 3525 3200
-Connection ~ 2375 3500
+Connection ~ 2600 2900
+Connection ~ 2600 3200
 Wire Wire Line
 	3425 2900 3425 2800
 Wire Wire Line
-	1900 3500 2375 3500
-Wire Wire Line
-	2850 3500 3950 3500
-Wire Wire Line
-	2850 2200 2850 2300
+	2600 2200 2600 2250
 Connection ~ 1775 5025
 $Comp
@@
 	1    0    0    -1
 $EndComp
+Connection ~ 2600 1425
+Wire Wire Line
+	2600 1425 3025 1425
+Wire Wire Line
+	2600 2900 3425 2900
+Wire Wire Line
+	2600 3200 3525 3200
+Wire Wire Line
+	2600 3500 3950 3500
+Connection ~ 3950 3500
+Wire Wire Line
+	2600 2200 3250 2200
+Wire Wire Line
+	1075 1425 1825 1425
+Wire Wire Line
+	1825 2200 1825 1425
+Wire Wire Line
+	1825 2600 1825 3500
+$Comp
+L formula:D_TVS_35V D?
+U 1 1 61F5EEBD
+P 1825 2600
+F 0 "D?" H 2075 2475 60  0000 R CNN
+F 1 "D_TVS_35V" H 2250 2725 60  0000 R CNN
+F 2 "SMC_DIO" H 2025 2240 60  0001 C CNN
+F 3 "https://www.diodes.com/assets/Datasheets/ds40741.pdf" H 1825 2600 60  0001 C CNN
+F 4 "SMCJ22A-13-F" H 1975 2850 50  0001 C CNN "MPN"
+	1    1825 2600
+	0    -1   -1   0
+$EndComp
+$Comp
+L formula:R_1.54K R?
+U 1 1 61D037A0
+P 2125 2400
+F 0 "R?" H 2195 2446 50  0000 L CNN
+F 1 "R_1.54K" H 2195 2355 50  0000 L CNN
+F 2 "footprints:R_0805_OEM" H 2055 2400 50  0001 C CNN
+F 3 "https://industrial.panasonic.com/cdbs/www-data/pdf/RDA0000/AOA0000C304.pdf" H 2205 2400 50  0001 C CNN
+F 4 "Panasonic" H 2125 2400 50  0001 C CNN "MFN"
+F 5 "ERJ-6ENF1541V" H 2125 2400 50  0001 C CNN "MPN"
+F 6 "https://www.digikey.com/en/products/detail/panasonic-electronic-components/ERJ-6ENF1541V/111317" H 2125 2400 50  0001 C CNN "Purchasing Link"
+	1    2125 2400
+	1    0    0    -1
+$EndComp
+$Comp
+L formula:R_500 U?
+U 1 1 61D01F28
+P 2125 2750
+F 0 "U?" V 2079 2838 50  0000 L CNN
+F 1 "R_500" V 2170 2838 50  0000 L CNN
+F 2 "footprints:R_0805_OEM" H 2125 2750 50  0001 C CNN
+F 3 "" H 2125 2750 50  0001 C CNN
+	1    2125 2750
+	0    1    1    0
+$EndComp
+Connection ~ 1825 1425
+Connection ~ 1825 3500
+Wire Wire Line
+	1825 3500 1900 3500
+Wire Wire Line
+	1825 1425 2600 1425
+Wire Wire Line
+	2125 2550 2125 2575
+Wire Wire Line
+	2125 2250 2600 2250
+Connection ~ 2600 2250
+Wire Wire Line
+	2600 2250 2600 2300
+Wire Wire Line
+	2125 2900 2125 3500
+Wire Wire Line
+	1900 3500 2125 3500
+Connection ~ 2125 3500
+Wire Wire Line
+	2125 3500 2600 3500
+Wire Wire Line
+	2125 2575 2225 2575
+Connection ~ 2125 2575
+Wire Wire Line
+	2125 2575 2125 2600
+Text Label 2225 2575 0    50   ~ 0
+SHDN
 $EndSCHEMATC
