File: bldc_foc_controller/bldc_foc_controller.sch (KiCad schematic (older format))
At the start: 157 parts

Commit message: minor changes
Parts:
- J1: renamed from J?; footprint (none) -> Connector_PinHeader_2.54mm:PinHeader_1x05_P2.54mm_Vertical
- gave numbers to parts that had none: 156

Commit message: layout changes
Parts:
- J2, J3: footprint (none) -> Connector_PinSocket_2.54mm:PinSocket_2x19_P2.54mm_Vertical_SMD
- J6: footprint Pin_Headers:Pin_Header_Straight_1x03_Pitch2.54mm -> Connector_PinHeader_2.54mm:PinHeader_1x03_P2.54mm_Vertical_SMD_Pin1Left
- L1: footprint (none) -> footprints:SRP0520-4R7K
Connections:
- net GND: no longer U4.15 (EPAD), U4.2 (SYNC), U4.3 (RO), U4.8 (PGND), U4.9 (PGND)
- net VBUS: no longer U4.5 (EN), U4.6 (VS), U4.7 (VS)
- net at U4.10 (SW), U4.11 (SW): no longer L1.1
- net at C7.2, NT1.2, R11.2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: no longer U4.12 (SSON), U4.4 (AGND)
- net at C6.2, R10.2, R11.1: no longer U4.14 (FB)
- net at R2.1: no longer U4.1 (FREQ)
- net at U4.13 (RT): no longer R9.1
- new net PGND: U4.8 (PGND), U4.9 (PGND)
- new net VS: U4.6 (VS), U4.7 (VS)
Other:
- moved on the sheet: U4
Changed lines of the file:
@@
 F 0 "J2" H 6900 6492 50  0000 C CNN
 F 1 "Conn_02x19_Odd_Even" H 6900 6401 50  0000 C CNN
-F 2 "" H 6850 5375 50  0001 C CNN
+F 2 "Connector_PinSocket_2.54mm:PinSocket_2x19_P2.54mm_Vertical_SMD" H 6850 5375 50  0001 C CNN
 F 3 "~" H 6850 5375 50  0001 C CNN
 	1    6850 5375
@@
 F 0 "J3" H 8750 6492 50  0000 C CNN
 F 1 "Conn_02x19_Odd_Even" H 8750 6401 50  0000 C CNN
-F 2 "" H 8700 5375 50  0001 C CNN
+F 2 "Connector_PinSocket_2.54mm:PinSocket_2x19_P2.54mm_Vertical_SMD" H 8700 5375 50  0001 C CNN
 F 3 "~" H 8700 5375 50  0001 C CNN
 	1    8700 5375
@@
 $EndComp
 $Comp
-L formula:CONN_01X03 J6
-U 1 1 618C4A73
-P 12800 9800
-F 0 "J6" V 12713 9612 50  0000 R CNN
-F 1 "CONN_01X03" V 12622 9612 50  0000 R CNN
-F 2 "Pin_Headers:Pin_Header_Straight_1x03_Pitch2.54mm" H 12800 8600 50  0001 C CNN
-F 3 "https://www.mouser.com/datasheet/2/181/M20-999-1218971.pdf" H 12800 8600 50  0001 C CNN
-F 4 "Mouser" H 12800 9800 60  0001 C CNN "MFN"
-F 5 "855-M20-9990346" H 12800 9800 60  0001 C CNN "MPN"
-F 6 "https://www.mouser.com/ProductDetail/Harwin/M20-9990346?qs=sGAEpiMZZMs%252bGHln7q6pmzlZUuX%2f53qj1ROyRKct5o4%3d" H 13200 10400 60  0001 C CNN "PurchasingLink"
-	1    12800 9800
-	0    -1   -1   0
-$EndComp
-$Comp
 L formula:CONN_01x02 J8
 U 1 1 618CA5DC
@@
 F 0 "L1" V 3525 5075 50  0000 C CNN
 F 1 "SRP0520-4R7K" V 3700 4900 50  0000 C CNN
-F 2 "" H 3600 5025 50  0001 C CNN
+F 2 "footprints:SRP0520-4R7K" H 3600 5025 50  0001 C CNN
 F 3 "https://www.bourns.com/docs/product-datasheets/srp0520.pdf" H 3600 5025 50  0001 C CNN
 	1    3600 5025
@@
 LTC4368 for Precharge, OV/UV\nProtection, Overcurrent & \nReverse Current Protection
 $Comp
-L Device:C C12
-U 1 1 61D36A19
-P 8125 1400
-F 0 "C12" V 7975 1350 50  0000 L CNN
-F 1 "C_10uF" V 8250 1250 50  0000 L CNN
-F 2 "footprints:C_1206_OEM" H 8163 1250 50  0001 C CNN
-F 3 "https://media.digikey.com/pdf/Data%20Sheets/Samsung%20PDFs/CL31A106KBHNNNE_Spec.pdf" H 8125 1400 50  0001 C CNN
-	1    8125 1400
-	1    0    0    -1
-$EndComp
-$Comp
 L Device:C C17
 U 1 1 61D41163
@@
 Wire Wire Line
 	8725 1550 8875 1550
-Text Notes 8350 1150 0    50   ~ 0
-1206 MLCC X5R Cap Bank\n10uF @50V \nDerates to 1.8uF @25V
 Wire Wire Line
 	9600 1250 10075 1250
@@
 $EndComp
 $Comp
-L Device:CP1 C35
-U 1 1 61ECCB07
-P 10875 1400
-F 0 "C35" V 10750 1350 50  0000 L CNN
-F 1 "C_100uF" V 11025 1200 50  0000 L CNN
-F 2 "Capacitor_THT:CP_Radial_D6.3mm_P2.50mm" H 10875 1400 50  0001 C CNN
-F 3 "" H 10875 1400 50  0001 C CNN
-F 4 "THT 6.3mm 35v 100uF 50mohm alpolys for 15c each" H 10875 1400 50  0001 C CNN "Desc"
-	1    10875 1400
-	1    0    0    -1
-$EndComp
-$Comp
 L Device:CP1 C36
 U 1 1 61ECCB0E
@@
 L formula:TLS4120D0EPVXUMA1 U4
 U 1 1 6198C5F2
-P 1775 5025
-F 0 "U4" H 2575 5312 60  0000 C CNN
-F 1 "TLS4120D0EPVXUMA1" H 2575 5206 60  0000 C CNN
-F 2 "footprints:TLS4120D0EPVXUMA1" H 2475 4125 60  0001 C CNN
-F 3 "https://www.infineon.com/dgdl/Infineon-TLS4120D0EPV-DataSheet-v01_00-EN.pdf?fileId=5546d46270c4f93e01710b576dc53b30" H 2575 5206 60  0001 C CNN
-	1    1775 5025
+P 14575 7100
+F 0 "U4" H 15375 7387 60  0000 C CNN
+F 1 "TLS4120D0EPVXUMA1" H 15375 7281 60  0000 C CNN
+F 2 "footprints:TLS4120D0EPVXUMA1" H 15275 6200 60  0001 C CNN
+F 3 "https://www.infineon.com/dgdl/Infineon-TLS4120D0EPV-DataSheet-v01_00-EN.pdf?fileId=5546d46270c4f93e01710b576dc53b30" H 15375 7281 60  0001 C CNN
+	1    14575 7100
 	1    0    0    -1
 $EndComp
@@
 Text Label 3600 2500 2    50   ~ 0
 ~SHDN
+$Comp
+L Device:CP1 C35
+U 1 1 61ECCB07
+P 10875 1400
+F 0 "C35" V 10750 1350 50  0000 L CNN
+F 1 "C_100uF" V 11025 1200 50  0000 L CNN
+F 2 "Capacitor_THT:CP_Radial_D6.3mm_P2.50mm" H 10875 1400 50  0001 C CNN
+F 3 "" H 10875 1400 50  0001 C CNN
+F 4 "THT 6.3mm 35v 100uF 50mohm alpolys for 15c each" H 10875 1400 50  0001 C CNN "Desc"
+	1    10875 1400
+	1    0    0    -1
+$EndComp
+Text Notes 8350 1150 0    50   ~ 0
+1206 MLCC X5R Cap Bank\n10uF @50V \nDerates to 1.8uF @25V
+$Comp
+L Device:C C12
+U 1 1 61D36A19
+P 8125 1400
+F 0 "C12" V 7975 1350 50  0000 L CNN
+F 1 "C_10uF" V 8250 1250 50  0000 L CNN
+F 2 "footprints:C_1206_OEM" H 8163 1250 50  0001 C CNN
+F 3 "https://media.digikey.com/pdf/Data%20Sheets/Samsung%20PDFs/CL31A106KBHNNNE_Spec.pdf" H 8125 1400 50  0001 C CNN
+	1    8125 1400
+	1    0    0    -1
+$EndComp
+$Comp
+L formula:CONN_01X03 J6
+U 1 1 618C4A73
+P 12800 9800
+F 0 "J6" V 12713 9612 50  0000 R CNN
+F 1 "CONN_01X03" V 12622 9612 50  0000 R CNN
+F 2 "Connector_PinHeader_2.54mm:PinHeader_1x03_P2.54mm_Vertical_SMD_Pin1Left" H 12800 8600 50  0000 C CNN
+F 3 "https://www.mouser.com/datasheet/2/181/M20-999-1218971.pdf" H 12800 8600 50  0001 C CNN
+F 4 "Mouser" H 12800 9800 60  0001 C CNN "MFN"
+F 5 "855-M20-9990346" H 12800 9800 60  0001 C CNN "MPN"
+F 6 "https://www.mouser.com/ProductDetail/Harwin/M20-9990346?qs=sGAEpiMZZMs%252bGHln7q6pmzlZUuX%2f53qj1ROyRKct5o4%3d" H 13200 10400 60  0001 C CNN "PurchasingLink"
+	1    12800 9800
+	0    -1   -1   0
+$EndComp
 $EndSCHEMATC

Commit message: Laying it out
Parts:
- J2, J3: footprint Connector_PinSocket_2.54mm:PinSocket_2x19_P2.54mm_Vertical_SMD -> Connector_PinSocket_2.54mm:PinSocket_2x19_P2.54mm_Vertical
- R1, R12, R24, R30, R36: footprint WSL2726_VIS -> formula:WSL27261L000FEB
Connections:
- net PGND is gone; now on net GND: U4.8 (PGND), U4.9 (PGND)
- net VS is gone; now on net VBUS: U4.6 (VS), U4.7 (VS)
- net GND: now also U4.15 (EPAD), U4.2 (SYNC), U4.3 (RO)
- net VBUS: now also U4.5 (EN)
- net at L1.1: now also U4.10 (SW), U4.11 (SW)
- net at C7.2, NT1.2, R11.2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: now also U4.12 (SSON), U4.4 (AGND)
- net at C6.2, R10.2, R11.1: now also U4.14 (FB)
- net at R2.1: now also U4.1 (FREQ)
- net at U4.13 (RT): now also R9.1
Other:
- moved on the sheet: U4
Changed lines of the file:
@@
 F 0 "J2" H 6900 6492 50  0000 C CNN
 F 1 "Conn_02x19_Odd_Even" H 6900 6401 50  0000 C CNN
-F 2 "Connector_PinSocket_2.54mm:PinSocket_2x19_P2.54mm_Vertical_SMD" H 6850 5375 50  0001 C CNN
+F 2 "Connector_PinSocket_2.54mm:PinSocket_2x19_P2.54mm_Vertical" H 6850 5375 50  0001 C CNN
 F 3 "~" H 6850 5375 50  0001 C CNN
 	1    6850 5375
@@
 F 0 "J3" H 8750 6492 50  0000 C CNN
 F 1 "Conn_02x19_Odd_Even" H 8750 6401 50  0000 C CNN
-F 2 "Connector_PinSocket_2.54mm:PinSocket_2x19_P2.54mm_Vertical_SMD" H 8700 5375 50  0001 C CNN
+F 2 "Connector_PinSocket_2.54mm:PinSocket_2x19_P2.54mm_Vertical" H 8700 5375 50  0001 C CNN
 F 3 "~" H 8700 5375 50  0001 C CNN
 	1    8700 5375
@@
 F 0 "R12" H 4800 1475 60  0000 C CNN
 F 1 "R_1m_3W_1%" H 4825 1698 60  0000 C CNN
-F 2 "WSL2726_VIS" H 4775 1140 60  0001 C CNN
+F 2 "formula:WSL27261L000FEB" H 4775 1140 60  0001 C CNN
 F 3 "https://www.vishay.com/docs/30131/wsl2726.pdf" H 4525 1475 60  0001 C CNN
 F 4 "WSL27261L000FEB" H 4825 975 50  0001 C CNN "MPN"
@@
 F 0 "R1" H 1350 1175 60  0000 C CNN
 F 1 "R_1m_3W_1%" H 1375 1398 60  0000 C CNN
-F 2 "WSL2726_VIS" H 1325 840 60  0001 C CNN
+F 2 "formula:WSL27261L000FEB" H 1325 840 60  0001 C CNN
 F 3 "https://www.vishay.com/docs/30131/wsl2726.pdf" H 1075 1175 60  0001 C CNN
 F 4 "WSL27261L000FEB" H 1375 675 50  0001 C CNN "MPN"
@@
 Wire Wire Line
 	2600 2200 2600 2250
-Connection ~ 1775 5025
 $Comp
 L formula:TLS4120D0EPVXUMA1 U4
 U 1 1 6198C5F2
-P 14575 7100
-F 0 "U4" H 15375 7387 60  0000 C CNN
-F 1 "TLS4120D0EPVXUMA1" H 15375 7281 60  0000 C CNN
-F 2 "footprints:TLS4120D0EPVXUMA1" H 15275 6200 60  0001 C CNN
-F 3 "https://www.infineon.com/dgdl/Infineon-TLS4120D0EPV-DataSheet-v01_00-EN.pdf?fileId=5546d46270c4f93e01710b576dc53b30" H 15375 7281 60  0001 C CNN
-	1    14575 7100
+P 1775 5025
+F 0 "U4" H 2575 5312 60  0000 C CNN
+F 1 "TLS4120D0EPVXUMA1" H 2575 5206 60  0000 C CNN
+F 2 "footprints:TLS4120D0EPVXUMA1" H 2475 4125 60  0001 C CNN
+F 3 "https://www.infineon.com/dgdl/Infineon-TLS4120D0EPV-DataSheet-v01_00-EN.pdf?fileId=5546d46270c4f93e01710b576dc53b30" H 2575 5206 60  0001 C CNN
+	1    1775 5025
 	1    0    0    -1
 $EndComp
@@
 	1650 5575 1775 5575
 Wire Wire Line
-	2425 6125 2500 6125
-Wire Wire Line
 	2325 6125 2400 6125
-Connection ~ 2425 6125
 Wire Wire Line
 	3525 6375 2400 6375
 Connection ~ 2400 6125
 Wire Wire Line
-	2400 6125 2425 6125
-Wire Wire Line
 	1150 5675 1325 5675
 Wire Wire Line
@@
 Text Notes 775  10650 0    50   ~ 0
 Unidirectional TVS \ndiodes for ESD protection
-Wire Wire Line
-	2700 6125 2775 6125
-Connection ~ 2775 6125
-Wire Wire Line
-	2775 6125 2975 6125
 $Comp
 L power:GND #PWR0161
@@
 F 0 "R36" H 16900 6800 60  0000 C CNN
 F 1 "R_1m_3W_1%" H 16900 7023 60  0000 C CNN
-F 2 "WSL2726_VIS" H 16850 6465 60  0001 C CNN
+F 2 "formula:WSL27261L000FEB" H 16850 6465 60  0001 C CNN
 F 3 "https://www.vishay.com/docs/30131/wsl2726.pdf" H 16600 6800 60  0001 C CNN
 F 4 "WSL27261L000FEB" H 16900 6300 50  0001 C CNN "MPN"
@@
 F 0 "R30" H 14650 6800 60  0000 C CNN
 F 1 "R_1m_3W_1%" H 14650 7023 60  0000 C CNN
-F 2 "WSL2726_VIS" H 14600 6465 60  0001 C CNN
+F 2 "formula:WSL27261L000FEB" H 14600 6465 60  0001 C CNN
 F 3 "https://www.vishay.com/docs/30131/wsl2726.pdf" H 14350 6800 60  0001 C CNN
 F 4 "WSL27261L000FEB" H 14650 6300 50  0001 C CNN "MPN"
@@
 F 0 "R24" H 12250 6800 60  0000 C CNN
 F 1 "R_1m_3W_1%" H 12250 7023 60  0000 C CNN
-F 2 "WSL2726_VIS" H 12200 6465 60  0001 C CNN
+F 2 "formula:WSL27261L000FEB" H 12200 6465 60  0001 C CNN
 F 3 "https://www.vishay.com/docs/30131/wsl2726.pdf" H 11950 6800 60  0001 C CNN
 F 4 "WSL27261L000FEB" H 12250 6300 50  0001 C CNN "MPN"
@@
 	0    -1   -1   0
 $EndComp
+Wire Wire Line
+	2400 6125 2425 6125
+Wire Wire Line
+	2700 6125 2775 6125
+Connection ~ 2775 6125
+Wire Wire Line
+	2775 6125 2975 6125
+Connection ~ 2425 6125
+Wire Wire Line
+	2425 6125 2500 6125
+Connection ~ 1775 5025
 $EndSCHEMATC
