File: bldc_foc_controller/bldc_foc_controller.sch (KiCad schematic (older format))
At the start: 194 parts, among them J1 Conn_01x05, J2 Conn_02x19_Odd_Even, J3 Conn_02x19_Odd_Even, J4 Conn_01x10, J6 CONN_01X03, J7 CONN_01x02, J8 CONN_01x02, Q1 HYG025N06LS1C2, Q10 PSMN2R2-40YSD, Q11 DNP, Q12 DNP, Q13 PSMN2R2-40YSD, Q14 PSMN2R2-40YSD, Q15 DNP, Q16 DNP, Q2 HYG025N06LS1C2, Q3 HYG025N06LS1C2, Q4 HYG025N06LS1C2, Q5 PSMN2R2-40YSD, Q6 PSMN2R2-40YSD, Q7 DNP, Q8 DNP, Q9 PSMN2R2-40YSD, U1 redcube-7461057, U10 INA240A1D, U11 INA240A1D, U12 DRV8320S, U13 INA240A1D, U2 redcube-7461057, U3 redcube-7461057, U4 TLS4120D0EPVXUMA1, U5 R_500, U6 redcube-7461057, U7 LTC4368CMS-1-PBF, U8 LMP8481ASQDGKRQ1, U9 LMP8481ASQDGKRQ1

Commit message: fixing merge errors
Parts:
- added C?: C_100nF, footprints:C_0603_1608Metric, symbol formula:C_100nF
- added C?: C_10uF_50V, footprints:C_0805_OEM, symbol formula:C_10uF_50V
- added J?: CONN_01x02, footprints:PinHeader_1x02_P2.54mm_Vertical, symbol formula:CONN_01x02
Connections:
- net GND: now also C55.1, NT2.1, U12.31 (PGND), C?.1, C?.1
- net INHA: now also J?.2 (Pin_2)
- net VBUS: now also C45.1, C?.2, C?.2
- net at J6.1 (P1): now also J?.1 (Pin_1)
- net at U12.1 (CPH): now also C50.2
- net at U12.2 (VCP): now also C45.2
- net at U12.32 (CPL): now also C50.1
Changed lines of the file:
@@
 	17675 1950 17750 1950
-Wire Wire Line
-	16825 1450 16975 1450
 Wire Wire Line
 	17100 1450 17100 1350
@@
 	1    0    0    -1
 $EndComp
-Wire Wire Line
-	15050 1750 15300 1750
 Wire Wire Line
 	15300 1750 15300 1650
@@
 Wire Wire Line
 	8000 1250 8125 1250
-Wire Wire Line
-	15125 1450 15775 1450
-Wire Wire Line
-	15050 1450 15125 1450
-Connection ~ 15125 1450
 $Comp
 L formula:VBUS_20V #PWR0148
 U 1 1 67E5888A
-P 15125 1450
-F 0 "#PWR0148" H 15125 1300 50  0001 C CNN
-F 1 "VBUS_20V" H 15140 1623 50  0000 C CNN
-F 2 "" H 15125 1450 50  0001 C CNN
-F 3 "" H 15125 1450 50  0001 C CNN
-	1    15125 1450
+P 14975 1425
+F 0 "#PWR0148" H 14975 1275 50  0001 C CNN
+F 1 "VBUS_20V" H 14990 1598 50  0000 C CNN
+F 2 "" H 14975 1425 50  0001 C CNN
+F 3 "" H 14975 1425 50  0001 C CNN
+	1    14975 1425
 	1    0    0    -1
 $EndComp
@@
 Wire Notes Line
 	14625 9300 18750 9300
+Wire Wire Line
+	16525 1000 15775 1000
+Wire Wire Line
+	15775 1000 15775 1350
+Wire Wire Line
+	16825 1000 16825 1350
+Wire Wire Line
+	16825 1450 17100 1450
+Wire Wire Line
+	17100 1350 17150 1350
+Connection ~ 17150 1350
+Wire Wire Line
+	17150 1350 17200 1350
+Connection ~ 17250 1350
+Wire Wire Line
+	17250 1350 17750 1350
+$Comp
+L formula:CONN_01x02 J?
+U 1 1 61AF1248
+P 12425 10200
+F 0 "J?" H 12375 10325 50  0000 L CNN
+F 1 "CONN_01x02" H 12250 10000 50  0000 L CNN
+F 2 "footprints:PinHeader_1x02_P2.54mm_Vertical" H 12325 10200 50  0001 C CNN
+F 3 "https://katalog.we-online.de/em/datasheet/6130xx11121.pdf" H 12425 10300 50  0001 C CNN
+F 4 "DK" H 12525 10400 50  0001 C CNN "MFN"
+F 5 "732-5315-ND" H 12625 10500 50  0001 C CNN "MPN"
+	1    12425 10200
+	-1   0    0    1
+$EndComp
+Wire Wire Line
+	12700 10050 12700 10200
+Wire Wire Line
+	12700 10200 12625 10200
+Wire Wire Line
+	12625 10100 12625 9850
+Wire Wire Line
+	12625 9850 12600 9850
+Wire Wire Line
+	14975 1750 15300 1750
+Wire Wire Line
+	14975 1425 14975 1450
+Wire Wire Line
+	14975 1450 15275 1450
+Connection ~ 14975 1450
+Wire Wire Line
+	15375 900  17200 900
+Wire Wire Line
+	17200 900  17200 1350
+Connection ~ 17200 1350
+Wire Wire Line
+	17200 1350 17250 1350
+$Comp
+L formula:C_100nF C?
+U 1 1 61CFB379
+P 15475 1300
+F 0 "C?" H 15500 1375 50  0000 L CNN
+F 1 "C_100nF" H 15400 1500 50  0000 L CNN
+F 2 "footprints:C_0603_1608Metric" H 15513 1150 50  0001 C CNN
+F 3 "http://www.samsungsem.com/kr/support/product-search/mlcc/CL10A475KQ8NNNC.jsp" H 15500 1400 50  0001 C CNN
+F 4 "DK" H 15475 1300 60  0001 C CNN "MFN"
+F 5 "1276-6717-1-ND" H 15475 1300 60  0001 C CNN "MPN"
+F 6 "https://www.digikey.com/product-detail/en/samsung-electro-mechanics/CL10B104KA8WPNC/1276-6717-1-ND/5961576" H 15900 1800 60  0001 C CNN "PurchasingLink"
+	1    15475 1300
+	1    0    0    -1
+$EndComp
+Connection ~ 15475 1450
+Wire Wire Line
+	15475 1450 15775 1450
+$Comp
+L formula:C_10uF_50V C?
+U 1 1 61D53CF1
+P 15275 1350
+F 0 "C?" H 15300 1475 50  0000 L CNN
+F 1 "C_10uF_50V" H 14900 1600 50  0000 L CNN
+F 2 "footprints:C_0805_OEM" H 15313 1950 50  0001 C CNN
+F 3 "http://www.samsungsem.com/kr/support/product-https://search.murata.co.jp/Ceramy/image/img/A01X/G101/ENG/GRM21BR61H106KE43-01A.pdf" H 15300 2200 50  0001 C CNN
+F 4 "Murata" H 15275 1400 60  0001 C CNN "MFN"
+F 5 "GRM21BR61H106KE43L" H 15275 2100 60  0001 C CNN "MPN"
+F 6 "https://www.digikey.com/en/products/detail/murata-electronics/GRM21BR61H106KE43L/10326316" H 15700 1850 60  0001 C CNN "PurchasingLink"
+	1    15275 1350
+	1    0    0    -1
+$EndComp
+Connection ~ 15275 1450
+Wire Wire Line
+	15275 1450 15475 1450
+Wire Wire Line
+	15375 1150 15475 1150
+Wire Wire Line
+	15375 900  15375 1150
+Wire Wire Line
+	15275 1150 15375 1150
+Connection ~ 15375 1150
 $EndSCHEMATC

Commit message: additional merge fixes
Connections:
- net GND: no longer C55.1, C?.1, C?.1, NT2.1, U12.31 (PGND)
- net at U12.23 (AGND): now also NT2.1
- new net: C55.1, C?.1, C?.1, U12.31 (PGND)
Other:
- moved on the sheet: NT2
Changed lines of the file:
@@
 L Device:Net-Tie_2 NT2
 U 1 1 670E9C37
-P 17250 1450
-F 0 "NT2" V 17250 1631 50  0000 C CNN
-F 1 "Net-Tie_2" V 17200 1650 50  0000 C CNN
-F 2 "" H 17250 1450 50  0001 C CNN
-F 3 "~" H 17250 1450 50  0001 C CNN
-	1    17250 1450
+P 17600 1650
+F 0 "NT2" V 17600 1831 50  0000 C CNN
+F 1 "Net-Tie_2" V 17550 1850 50  0000 C CNN
+F 2 "" H 17600 1650 50  0001 C CNN
+F 3 "~" H 17600 1650 50  0001 C CNN
+	1    17600 1650
 	0    1    1    0
-$EndComp
-$Comp
-L power:GND #PWR0145
-U 1 1 671C9CD5
-P 17150 1350
-F 0 "#PWR0145" H 17150 1100 50  0001 C CNN
-F 1 "GND" H 17155 1177 50  0000 C CNN
-F 2 "" H 17150 1350 50  0001 C CNN
-F 3 "" H 17150 1350 50  0001 C CNN
-	1    17150 1350
-	1    0    0    -1
 $EndComp
 Text Label 17000 1950 0    50   ~ 0
@@
 	17750 1350 17750 1650
 Wire Wire Line
-	17600 1950 17600 1550
-Wire Wire Line
-	17600 1550 17250 1550
+	17600 1950 17600 1750
 Connection ~ 17600 1950
 Wire Wire Line
@@
 Wire Wire Line
 	16825 1450 17100 1450
-Wire Wire Line
-	17100 1350 17150 1350
-Connection ~ 17150 1350
-Wire Wire Line
-	17150 1350 17200 1350
-Connection ~ 17250 1350
-Wire Wire Line
-	17250 1350 17750 1350
 $Comp
 L formula:CONN_01x02 J?
@@
 	17200 900  17200 1350
 Connection ~ 17200 1350
-Wire Wire Line
-	17200 1350 17250 1350
 $Comp
 L formula:C_100nF C?
@@
 	15275 1150 15375 1150
 Connection ~ 15375 1150
+Wire Wire Line
+	17100 1350 17200 1350
+Wire Wire Line
+	17200 1350 17750 1350
+Wire Wire Line
+	16825 1550 17600 1550
 $EndSCHEMATC

Commit message: more layout, ay
Parts:
- C61: renamed from C?; footprint footprints:C_0805_OEM -> formula:C_0805_OEM
- C62: renamed from C?; footprint footprints:C_0603_1608Metric -> formula:C_0603_1608Metric
- H1, H2, H3: footprint (none) -> TestPoint:TestPoint_Pad_4.0x4.0mm
- gave numbers to parts that had none: 5
Changed lines of the file:
@@
 F 0 "H1" V 1150 9575 50  0000 C CNN
 F 1 "MotorConnector_Pad" V 1050 9525 50  0000 C CNN
-F 2 "" H 925 9675 50  0001 C CNN
+F 2 "TestPoint:TestPoint_Pad_4.0x4.0mm" H 925 9675 50  0001 C CNN
 F 3 "~" H 925 9675 50  0001 C CNN
 	1    925  9675
@@
 F 0 "H2" V 1150 9900 50  0000 C CNN
 F 1 "MotorConnector_Pad" V 1050 9850 50  0000 C CNN
-F 2 "" H 925 10000 50  0001 C CNN
+F 2 "TestPoint:TestPoint_Pad_4.0x4.0mm" H 925 10000 50  0001 C CNN
 F 3 "~" H 925 10000 50  0001 C CNN
 	1    925  10000
@@
 F 0 "H3" V 1150 10225 50  0000 C CNN
 F 1 "MotorConnector_Pad" V 1050 10175 50  0000 C CNN
-F 2 "" H 925 10325 50  0001 C CNN
+F 2 "TestPoint:TestPoint_Pad_4.0x4.0mm" H 925 10325 50  0001 C CNN
 F 3 "~" H 925 10325 50  0001 C CNN
 	1    925  10325
@@
 	17125 9050 17125 9100
 $Comp
-L formula:LED_0805 D?
+L formula:LED_0805 D10
 U 1 1 63061182
 P 15725 8600
-F 0 "D?" V 15775 8825 50  0000 R CNN
+F 0 "D10" V 15775 8825 50  0000 R CNN
 F 1 "LED_0805" V 15675 9050 50  0000 R CNN
 F 2 "footprints:LED_0805_OEM" H 15625 8600 50  0001 C CNN
@@
 $EndComp
 $Comp
-L Device:R R?
+L Device:R R50
 U 1 1 63061188
 P 15725 8900
-F 0 "R?" H 15500 8975 50  0000 L CNN
+F 0 "R50" H 15500 8975 50  0000 L CNN
 F 1 "R_68" H 15400 8850 50  0000 L CNN
 F 2 "footprints:R_0805_OEM" V 15655 8900 50  0001 C CNN
@@
 $EndComp
 $Comp
-L power:GND #PWR?
+L power:GND #PWR0145
 U 1 1 6306118E
 P 15725 9100
-F 0 "#PWR?" H 15725 8850 50  0001 C CNN
+F 0 "#PWR0145" H 15725 8850 50  0001 C CNN
 F 1 "GND" H 15600 9025 50  0000 C CNN
 F 2 "" H 15725 9100 50  0001 C CNN
@@
 	15725 9050 15725 9100
 $Comp
-L formula:LED_0805 D?
+L formula:LED_0805 D9
 U 1 1 630B6073
 P 15125 8600
-F 0 "D?" V 15175 8825 50  0000 R CNN
+F 0 "D9" V 15175 8825 50  0000 R CNN
 F 1 "LED_0805" V 15075 9050 50  0000 R CNN
 F 2 "footprints:LED_0805_OEM" H 15025 8600 50  0001 C CNN
@@
 $EndComp
 $Comp
-L Device:R R?
+L Device:R R49
 U 1 1 630B6079
 P 15125 8900
-F 0 "R?" H 14900 8975 50  0000 L CNN
+F 0 "R49" H 14900 8975 50  0000 L CNN
 F 1 "R_68" H 14800 8850 50  0000 L CNN
 F 2 "footprints:R_0805_OEM" V 15055 8900 50  0001 C CNN
@@
 $EndComp
 $Comp
-L power:GND #PWR?
+L power:GND #PWR0162
 U 1 1 630B607F
 P 15125 9100
-F 0 "#PWR?" H 15125 8850 50  0001 C CNN
+F 0 "#PWR0162" H 15125 8850 50  0001 C CNN
 F 1 "GND" H 15000 9025 50  0000 C CNN
 F 2 "" H 15125 9100 50  0001 C CNN
@@
 	16825 1450 17100 1450
 $Comp
-L formula:CONN_01x02 J?
+L formula:CONN_01x02 J5
 U 1 1 61AF1248
 P 12425 10200
-F 0 "J?" H 12375 10325 50  0000 L CNN
+F 0 "J5" H 12375 10325 50  0000 L CNN
 F 1 "CONN_01x02" H 12250 10000 50  0000 L CNN
 F 2 "footprints:PinHeader_1x02_P2.54mm_Vertical" H 12325 10200 50  0001 C CNN
@@
 Connection ~ 17200 1350
 $Comp
-L formula:C_100nF C?
+L formula:C_100nF C62
 U 1 1 61CFB379
 P 15475 1300
-F 0 "C?" H 15500 1375 50  0000 L CNN
+F 0 "C62" H 15500 1375 50  0000 L CNN
 F 1 "C_100nF" H 15400 1500 50  0000 L CNN
-F 2 "footprints:C_0603_1608Metric" H 15513 1150 50  0001 C CNN
+F 2 "formula:C_0603_1608Metric" H 15513 1150 50  0001 C CNN
 F 3 "http://www.samsungsem.com/kr/support/product-search/mlcc/CL10A475KQ8NNNC.jsp" H 15500 1400 50  0001 C CNN
 F 4 "DK" H 15475 1300 60  0001 C CNN "MFN"
@@
 	15475 1450 15775 1450
 $Comp
-L formula:C_10uF_50V C?
+L formula:C_10uF_50V C61
 U 1 1 61D53CF1
 P 15275 1350
-F 0 "C?" H 15300 1475 50  0000 L CNN
+F 0 "C61" H 15300 1475 50  0000 L CNN
 F 1 "C_10uF_50V" H 14900 1600 50  0000 L CNN
-F 2 "footprints:C_0805_OEM" H 15313 1950 50  0001 C CNN
+F 2 "formula:C_0805_OEM" H 15313 1950 50  0001 C CNN
 F 3 "http://www.samsungsem.com/kr/support/product-https://search.murata.co.jp/Ceramy/image/img/A01X/G101/ENG/GRM21BR61H106KE43-01A.pdf" H 15300 2200 50  0001 C CNN
 F 4 "Murata" H 15275 1400 60  0001 C CNN "MFN"

Commit message: layout pushing
Parts:
- renumbered U5 to R51
Changed lines of the file:
@@
 $EndComp
 $Comp
-L formula:R_500 U5
+L formula:R_500 R51
 U 1 1 61D01F28
 P 2125 2750
-F 0 "U5" V 2079 2838 50  0000 L CNN
+F 0 "R51" V 2079 2838 50  0000 L CNN
 F 1 "R_500" V 2170 2838 50  0000 L CNN
 F 2 "footprints:R_0805_OEM" H 2125 2750 50  0001 C CNN

Commit message: schem changes, layout changes
Parts:
- C61: footprint formula:C_0805_OEM -> footprints:C_0805_OEM
- C62: footprint formula:C_0603_1608Metric -> footprints:C_0805_OEM
- C9: footprint footprints:C_100uF+ -> footprints:C_0805_OEM
- D1, D2, D3, D4, D5: footprint SMC_DIO -> footprints:DO-214AB
- U1, U2, U3, U6: footprint formula:redcube_pressfit_6pin -> footprints:redcube_pressfit_6pin
Changed lines of the file:
@@
 F 0 "U6" H 2400 1075 50  0000 L CNN
 F 1 "redcube-7461057" H 2100 1150 50  0000 L CNN
-F 2 "formula:redcube_pressfit_6pin" H 2425 1075 50  0001 C CNN
+F 2 "footprints:redcube_pressfit_6pin" H 2425 1075 50  0001 C CNN
 F 3 "https://www.mouser.com/datasheet/2/445/7461057-1723744.pdf" H 2425 1075 50  0001 C CNN
 F 4 "7461057" H 2425 1075 50  0001 C CNN "MPN"
@@
 F 0 "U3" V 1071 3638 50  0000 L CNN
 F 1 "redcube-7461057" V 1300 3500 50  0000 L CNN
-F 2 "formula:redcube_pressfit_6pin" H 1175 3650 50  0001 C CNN
+F 2 "footprints:redcube_pressfit_6pin" H 1175 3650 50  0001 C CNN
 F 3 "https://www.mouser.com/datasheet/2/445/7461057-1723744.pdf" H 1175 3650 50  0001 C CNN
 F 4 "7461057" H 1175 3650 50  0001 C CNN "MPN"
@@
 F 0 "U1" V 571 1513 50  0000 L CNN
 F 1 "redcube-7461057" V 675 1500 50  0000 L CNN
-F 2 "formula:redcube_pressfit_6pin" H 675 1525 50  0001 C CNN
+F 2 "footprints:redcube_pressfit_6pin" H 675 1525 50  0001 C CNN
 F 3 "https://www.mouser.com/datasheet/2/445/7461057-1723744.pdf" H 675 1525 50  0001 C CNN
 F 4 "7461057" H 675 1525 50  0001 C CNN "MPN"
@@
 F 0 "U2" V 571 3588 50  0000 L CNN
 F 1 "redcube-7461057" V 675 2750 50  0000 L CNN
-F 2 "formula:redcube_pressfit_6pin" H 675 3600 50  0001 C CNN
+F 2 "footprints:redcube_pressfit_6pin" H 675 3600 50  0001 C CNN
 F 3 "https://www.mouser.com/datasheet/2/445/7461057-1723744.pdf" H 675 3600 50  0001 C CNN
 F 4 "7461057" H 675 3600 50  0001 C CNN "MPN"
@@
 F 0 "C9" H 5440 1771 50  0000 L CNN
 F 1 "C_100uF+" H 5440 1680 50  0000 L CNN
-F 2 "footprints:C_100uF+" H 5363 2275 50  0001 C CNN
+F 2 "footprints:C_0805_OEM" H 5363 2275 50  0001 C CNN
 F 3 "https://www.nichicon.co.jp/english/products/pdfs/e-uuq.pdf" H 5350 2525 50  0001 C CNN
 F 4 "https://www.digikey.com/product-detail/en/nichicon/UUQ1H101MCL1GS/493-3209-2-ND/1965345" H 5750 2175 60  0001 C CNN "PurchasingLink"
@@
 Connection ~ 3575 1775
 Wire Wire Line
-	3775 1475 3825 1475
-Wire Wire Line
-	3825 1475 3825 925
-Wire Wire Line
-	3775 925  3825 925
-Connection ~ 3825 1475
-Wire Wire Line
-	3825 1475 3875 1475
-Connection ~ 3825 925
-Wire Wire Line
-	3825 925  3875 925
-Wire Wire Line
 	3500 1775 3575 1775
-Wire Wire Line
-	4075 1225 3875 1225
-Connection ~ 3875 1775
-Wire Wire Line
-	3875 1775 4075 1775
-Wire Wire Line
-	3575 1775 3775 1775
-Wire Wire Line
-	3575 1225 3775 1225
-Connection ~ 3775 1775
-Wire Wire Line
-	3775 1775 3875 1775
 $Comp
 L formula:C_100nF C2
@@
 Wire Wire Line
 	11275 10725 11325 10725
-Wire Wire Line
-	3875 1225 3875 1775
-Wire Wire Line
-	3775 1225 3775 1775
 $Comp
 L formula:R_1 R22
@@
 F 0 "D5" V 6103 2346 60  0000 R CNN
 F 1 "D_TVS_35V" H 6250 2575 60  0000 R CNN
-F 2 "SMC_DIO" H 6050 2090 60  0001 C CNN
+F 2 "footprints:DO-214AB" H 6050 2090 60  0001 C CNN
 F 3 "https://www.diodes.com/assets/Datasheets/ds40741.pdf" H 5850 2450 60  0001 C CNN
 F 4 "SMCJ22A-13-F" H 6000 2700 50  0001 C CNN "MPN"
@@
 F 0 "D2" H 2275 10025 60  0000 R CNN
 F 1 "D_TVS_35V" V 2475 10000 60  0000 R CNN
-F 2 "SMC_DIO" H 2100 9715 60  0001 C CNN
+F 2 "footprints:DO-214AB" H 2100 9715 60  0001 C CNN
 F 3 "https://www.diodes.com/assets/Datasheets/ds40741.pdf" H 1900 10075 60  0001 C CNN
 F 4 "SMCJ22A-13-F" H 2050 10325 50  0001 C CNN "MPN"
@@
 F 0 "D3" H 2475 10350 60  0000 R CNN
 F 1 "D_TVS_35V" V 2900 10525 60  0000 R CNN
-F 2 "SMC_DIO" H 2300 10040 60  0001 C CNN
+F 2 "footprints:DO-214AB" H 2300 10040 60  0001 C CNN
 F 3 "https://www.diodes.com/assets/Datasheets/ds40741.pdf" H 2100 10400 60  0001 C CNN
 F 4 "SMCJ22A-13-F" H 2250 10650 50  0001 C CNN "MPN"
@@
 F 0 "D4" H 2725 10675 60  0000 R CNN
 F 1 "D_TVS_35V" V 3375 11100 60  0000 R CNN
-F 2 "SMC_DIO" H 2550 10365 60  0001 C CNN
+F 2 "footprints:DO-214AB" H 2550 10365 60  0001 C CNN
 F 3 "https://www.diodes.com/assets/Datasheets/ds40741.pdf" H 2350 10725 60  0001 C CNN
 F 4 "SMCJ22A-13-F" H 2500 10975 50  0001 C CNN "MPN"
@@
 F 0 "D1" H 2075 2475 60  0000 R CNN
 F 1 "D_TVS_35V" H 2250 2725 60  0000 R CNN
-F 2 "SMC_DIO" H 2025 2240 60  0001 C CNN
+F 2 "footprints:DO-214AB" H 2025 2240 60  0001 C CNN
 F 3 "https://www.diodes.com/assets/Datasheets/ds40741.pdf" H 1825 2600 60  0001 C CNN
 F 4 "SMCJ22A-13-F" H 1975 2850 50  0001 C CNN "MPN"
@@
 F 0 "C62" H 15500 1375 50  0000 L CNN
 F 1 "C_100nF" H 15400 1500 50  0000 L CNN
-F 2 "formula:C_0603_1608Metric" H 15513 1150 50  0001 C CNN
+F 2 "footprints:C_0805_OEM" H 15513 1150 50  0001 C CNN
 F 3 "http://www.samsungsem.com/kr/support/product-search/mlcc/CL10A475KQ8NNNC.jsp" H 15500 1400 50  0001 C CNN
 F 4 "DK" H 15475 1300 60  0001 C CNN "MFN"
@@
 F 0 "C61" H 15300 1475 50  0000 L CNN
 F 1 "C_10uF_50V" H 14900 1600 50  0000 L CNN
-F 2 "formula:C_0805_OEM" H 15313 1950 50  0001 C CNN
+F 2 "footprints:C_0805_OEM" H 15313 1950 50  0001 C CNN
 F 3 "http://www.samsungsem.com/kr/support/product-https://search.murata.co.jp/Ceramy/image/img/A01X/G101/ENG/GRM21BR61H106KE43-01A.pdf" H 15300 2200 50  0001 C CNN
 F 4 "Murata" H 15275 1400 60  0001 C CNN "MFN"
@@
 Wire Wire Line
 	16825 1550 17600 1550
+Wire Wire Line
+	3775 1475 3800 1475
+Wire Wire Line
+	3775 925  3800 925
+Wire Wire Line
+	3575 1775 3850 1775
+Wire Wire Line
+	3575 1225 3850 1225
+Wire Wire Line
+	3850 1775 3850 1225
+Connection ~ 3850 1775
+Wire Wire Line
+	3850 1775 4075 1775
+Connection ~ 3850 1225
+Wire Wire Line
+	3850 1225 4075 1225
+Wire Wire Line
+	3800 1475 3800 925
+Connection ~ 3800 1475
+Wire Wire Line
+	3800 1475 3875 1475
+Connection ~ 3800 925
+Wire Wire Line
+	3800 925  3875 925
 $EndSCHEMATC

Commit message: still finishing inverter and other layouts
Parts:
- NT1: footprint (none) -> NetTie:NetTie-2_SMD_Pad0.5mm
Connections:
- net SYSTEM_SH_+: now also R12.3; no longer R12.2
- net SYSTEM_SH_-: now also R12.2; no longer R12.3
- net VBUS: now also R12.1; no longer R12.4
- net at Q3.1 (D), Q4.1 (D): now also R12.4; no longer R12.1
Changed lines of the file:
@@
 P 4075 1575
 F 0 "Q4" V 4300 1575 50  0000 C CNN
-F 1 "HYG025N06LS1C2" V 4800 2050 50  0000 C CNN
+F 1 "HYG025N06LS1C2" V 4950 1625 50  0000 C CNN
 F 2 "footprints:PDFN_5X6MC_MCH" H 4275 1675 50  0001 C CNN
 F 3 "https://drive.google.com/file/d/1Gbielo2qQ6OtCDVvoQN8r_uS-8EwH9-v/view?usp=sharing" H 4075 1575 50  0001 C CNN
@@
 P 4075 1025
 F 0 "Q3" V 4300 1025 50  0000 C CNN
-F 1 "HYG025N06LS1C2" V 4325 1500 50  0000 C CNN
+F 1 "HYG025N06LS1C2" V 4475 1075 50  0000 C CNN
 F 2 "footprints:PDFN_5X6MC_MCH" H 4275 1125 50  0001 C CNN
 F 3 "https://drive.google.com/file/d/1Gbielo2qQ6OtCDVvoQN8r_uS-8EwH9-v/view?usp=sharing" H 4075 1025 50  0001 C CNN
@@
 	10625 3600 18750 3600
 Connection ~ 1900 3500
-$Comp
-L formula:R_1m_3W_1% R12
-U 1 1 661E27D9
-P 4525 1475
-F 0 "R12" H 4800 1475 60  0000 C CNN
-F 1 "R_1m_3W_1%" H 4825 1698 60  0000 C CNN
-F 2 "formula:WSL27261L000FEB" H 4775 1140 60  0001 C CNN
-F 3 "https://www.vishay.com/docs/30131/wsl2726.pdf" H 4525 1475 60  0001 C CNN
-F 4 "WSL27261L000FEB" H 4825 975 50  0001 C CNN "MPN"
-	1    4525 1475
-	1    0    0    -1
-$EndComp
 Wire Wire Line
 	5125 1475 5325 1475
 Wire Wire Line
-	4350 925  4350 1475
-Connection ~ 4350 1475
-Wire Wire Line
-	4675 1475 4675 1800
-Wire Wire Line
-	4975 1800 4975 1475
+	4350 925  4350 975
 $Comp
 L formula:VBUS_20V #PWR0137
@@
 Wire Wire Line
 	1675 1175 2275 1175
-Text Label 4675 1700 2    50   ~ 0
+Text Label 4675 1800 1    50   ~ 0
 SYSTEM_SH_+
-Text Label 4950 2050 0    50   ~ 0
+Text Label 4950 1800 1    50   ~ 0
 SYSTEM_SH_-
 Wire Wire Line
 	4750 1800 4950 1800
 Wire Wire Line
-	4950 1800 4950 2050
-Connection ~ 4950 1800
-Wire Wire Line
-	4950 1800 4975 1800
-Wire Wire Line
 	4450 1800 4675 1800
-Wire Wire Line
-	4350 1475 4525 1475
 Wire Notes Line
 	14775 3200 14775 800
@@
 F 0 "NT1" H 3125 6250 50  0000 C CNN
 F 1 "Net-Tie_2" H 3000 6175 50  0000 C CNN
-F 2 "" H 3025 6100 50  0001 C CNN
+F 2 "NetTie:NetTie-2_SMD_Pad0.5mm" H 3025 6100 50  0001 C CNN
 F 3 "~" H 3025 6100 50  0001 C CNN
 	1    3025 6100
@@
 Wire Wire Line
 	3800 925  3875 925
+$Comp
+L formula:R_1m_3W_1% R12
+U 1 1 620B2503
+P 5100 975
+F 0 "R12" H 5375 975 60  0000 C CNN
+F 1 "R_1m_3W_1%" H 5400 1198 60  0000 C CNN
+F 2 "formula:WSL27261L000FEB" H 5350 640 60  0001 C CNN
+F 3 "https://www.vishay.com/docs/30131/wsl2726.pdf" H 5100 975 60  0001 C CNN
+F 4 "WSL27261L000FEB" H 5400 475 50  0001 C CNN "MPN"
+	1    5100 975
+	-1   0    0    1
+$EndComp
+Wire Wire Line
+	4500 975  4350 975
+Connection ~ 4350 975
+Wire Wire Line
+	4350 975  4350 1475
+Wire Wire Line
+	5100 975  5125 975
+Wire Wire Line
+	5125 975  5125 1475
+Text Label 4650 975  1    50   ~ 0
+SYSTEM_SH_+
+Text Label 4950 975  1    50   ~ 0
+SYSTEM_SH_-
 $EndSCHEMATC
