File: bldc_foc_controller/bldc_foc_controller.kicad_pcb (KiCad board)
At the start: 2 copper layers, 109.3 x 58.3 mm, 19 parts, among them U101 TPS560430YF

Commit message: layout changes
Parts:
- removed C101, C103: C_0.1uF, footprints:C_0805_OEM
- removed C102: C_2.2uF, footprints:C_0603_1608Metric
- removed COUT101: C_22uF, footprints:C_1206_OEM
- removed COUT102: C_33uF, footprints:Fuse_1812
- removed COUT103: C_47uF, footprints:C_0805_OEM
- removed D101: D_Zener_18V, footprints:DO-214AA
- removed D102, D103: LED_0805, footprints:LED_0805_OEM
- removed F101: F_500mA_16V, footprints:Fuse_1210
- removed G***: LOGO, footprints:Logo_Large
- removed G***: LOGO, footprints:phoenix
- removed L101: L_100uH, footprints:L_100uH_OEM
- removed R101: R_1K, footprints:R_0805_OEM
- removed R102: R_25K, footprints:R_0805_OEM
- removed R103: R_100K, footprints:R_0805_OEM
- removed R104: R_0_2512, footprints:R_2512_OEM
- removed R105: R_200, footprints:R_0805_OEM
- removed U101: TPS560430YF, footprints:SOT-23-6_OEM
- added C1: C_10uF, footprints:C_0805_OEM, F.Cu at (191.3, 90.7)
- added C10: C_10uF, footprints:C_0805_OEM, F.Cu at (122.7, 211.1)
- added C11: DNP, footprints:C_0805_OEM, F.Cu at (117.9, 253.7)
- added C12: C_10uF, footprints:C_1206_OEM, F.Cu at (77.5, 15.2)
- added C13: C_10uF, footprints:C_1206_OEM, F.Cu at (77.5, 18.5)
- added C14: C_10uF, footprints:C_1206_OEM, F.Cu at (77.4, 21.8)
- added C15: C_10uF, footprints:C_1206_OEM, F.Cu at (77.5, 25.1)
- added C16: C_10uF, footprints:C_0805_OEM, F.Cu at (142.5, 223.8)
- added C17: C_10uF, footprints:C_1206_OEM, F.Cu at (83.6, 15.2)
- added C18: C_10uF, footprints:C_1206_OEM, F.Cu at (83.6, 18.5)
- added C19: C_10uF, footprints:C_1206_OEM, F.Cu at (83.6, 21.8)
- added C2: C_100nF, footprints:C_0603_1608Metric, F.Cu at (119.1, 127.4)
- added C20: C_10uF, footprints:C_1206_OEM, F.Cu at (83.6, 25.1)
- added C21: DNP, footprints:C_0805_OEM, F.Cu at (117.9, 257.0)
- added C22: C_10uF, footprints:C_1206_OEM, F.Cu at (89.6, 15.2)
- added C23: C_10uF, footprints:C_1206_OEM, F.Cu at (89.6, 18.5)
- added C24: C_10uF, footprints:C_1206_OEM, F.Cu at (89.7, 21.8)
- added C25: C_10uF, footprints:C_1206_OEM, F.Cu at (89.6, 25.1)
- added C26: C_10uF, footprints:C_1206_OEM, F.Cu at (95.8, 15.2)
- added C27: C_10uF, footprints:C_1206_OEM, F.Cu at (95.8, 18.5)
- added C28: C_10uF, footprints:C_1206_OEM, F.Cu at (95.8, 21.8)
- added C29: C_10uF, footprints:C_1206_OEM, F.Cu at (95.8, 25.1)
- added C3: C_35nF, footprints:C_0805_OEM, F.Cu at (144.5, 127.0)
- added C30: C_10uF, footprints:C_0805_OEM, F.Cu at (154.2, 223.8)
- added C31: DNP, footprints:C_0805_OEM, F.Cu at (122.4, 257.0)
- added C32: C_100uF, Capacitor_THT:CP_Radial_D6.3mm_P2.50mm, F.Cu at (107.4, 17.0)
- added C33: C_10uF, footprints:C_0805_OEM, F.Cu at (165.9, 223.8)
- added C34: C_100uF, Capacitor_THT:CP_Radial_D6.3mm_P2.50mm, F.Cu at (115.1, 17.0)
- added C35: C_100uF, Capacitor_THT:CP_Radial_D6.3mm_P2.50mm, F.Cu at (123.2, 17.3)
- added C36: C_100uF, Capacitor_THT:CP_Radial_D6.3mm_P2.50mm, F.Cu at (130.8, 17.0)
- added C37: C_820uF, Capacitor_THT:CP_Radial_D8.0mm_P3.80mm, F.Cu at (154.2, 18.0)
- added C38: C_820uF, Capacitor_THT:CP_Radial_D8.0mm_P3.80mm, F.Cu at (144.8, 18.0)
- added C39: DNP, footprints:C_0805_OEM, F.Cu at (173.4, 104.6)
- added C4: C_10uF, footprints:C_0805_OEM, F.Cu at (168.8, 106.2)
- added C40: DNP, footprints:C_0805_OEM, F.Cu at (191.5, 87.9)
- added C41: C_10uF, footprints:C_1206_OEM, F.Cu at (175.2, 89.9)
- added C42: C_100nF, footprints:C_0805_OEM, F.Cu at (159.0, 120.0)
- added C43: C_10uF, footprints:C_1206_OEM, F.Cu at (175.4, 86.7)
- added C44: DNP, footprints:C_0805_OEM, F.Cu at (173.4, 107.4)
- added C45: C_1uF, footprints:C_0805_OEM, F.Cu at (184.1, 96.8)
- added C46: DNP, footprints:C_0805_OEM, F.Cu at (179.5, 99.7)
- added C47: DNP, footprints:C_0805_OEM, F.Cu at (153.6, 124.3)
- added C48: C_100nF, footprints:C_0805_OEM, F.Cu at (168.1, 113.0)
- added C49: C_10uF, footprints:C_1206_OEM, F.Cu at (152.7, 108.2)
- added C5: C_10uF, footprints:C_0805_OEM, F.Cu at (106.4, 211.1)
- added C50: C_47uF, footprints:C_0805_OEM, F.Cu at (177.9, 104.6)
- added C51: C_10uF, footprints:C_1206_OEM, F.Cu at (175.2, 93.0)
- added C52: DNP, footprints:C_0805_OEM, F.Cu at (149.0, 127.0)
- added C53: C_1uF, footprints:C_0805_OEM, F.Cu at (179.5, 96.8)
- added C54: C_100nF, footprints:C_0805_OEM, F.Cu at (163.6, 113.0)
- added C55: C_1uF, footprints:C_0805_OEM, F.Cu at (167.9, 110.2)
- added C56: DNP, footprints:C_0805_OEM, F.Cu at (185.7, 93.7)
- added C57: DNP, footprints:C_0805_OEM, F.Cu at (163.6, 115.8)
- added C58: DNP, footprints:C_0805_OEM, F.Cu at (153.5, 121.5)
- added C59: C_10uF, footprints:C_1206_OEM, F.Cu at (169.0, 99.2)
- added C6: C_10pF, footprints:C_0805_OEM, F.Cu at (114.8, 124.2)
- added C60: C_10uF, footprints:C_1206_OEM, F.Cu at (180.7, 89.9)
- added C7: C_220nF, footprints:C_0805_OEM, F.Cu at (159.0, 114.3)
- added C8: C_220nF, footprints:C_0805_OEM, F.Cu at (193.3, 81.9)
- added C9: C_100uF+, footprints:C_100uF+, F.Cu at (83.6, 77.5)
- added J1: Conn_01x05, Connector_PinHeader_2.54mm:PinHeader_1x05_P2.54mm_Vertical, F.Cu at (98.0, 251.2)
- added J2: Conn_02x19_Odd_Even, Connector_PinSocket_2.54mm:PinSocket_2x19_P2.54mm_Vertical_SMD, F.Cu at (-14.2, 136.4)
- added J3: Conn_02x19_Odd_Even, Connector_PinSocket_2.54mm:PinSocket_2x19_P2.54mm_Vertical_SMD, F.Cu at (-4.12, 136.4)
- added J4: Conn_01x10, footprints:PinHeader_1x10_P2.54mm_Vertical, F.Cu at (174.8, 207.8)
- added J5: CONN_01x02, footprints:PinHeader_1x02_P2.54mm_Vertical, F.Cu at (185.4, 209.0)
- added J6: CONN_01X03, Connector_PinHeader_2.54mm:PinHeader_1x03_P2.54mm_Vertical_SMD_Pin1Left, F.Cu at (190.5, 219.2)
- added J7: CONN_01x02, footprints:PinHeader_1x02_P2.54mm_Vertical, F.Cu at (190.8, 209.0)
- added J8: CONN_01x02, footprints:PinHeader_1x02_P2.54mm_Vertical, F.Cu at (196.1, 209.0)
- added L1: SRP0520-4R7K, footprints:SRP0520-4R7K, F.Cu at (34.2, 74.4)
- added Q1: HYG025N06LS1C2, footprints:PDFN_5X6MC_MCH, F.Cu at (121.8, 99.9)
- added Q10: PSMN2R2-40YSD, footprints:LFPAK56, F.Cu at (146.0, 106.1)
- added Q11: DNP, footprints:LFPAK56, F.Cu at (160.7, 91.4)
- added Q12: DNP, footprints:LFPAK56, F.Cu at (153.8, 103.6)
- added Q13: PSMN2R2-40YSD, footprints:LFPAK56, F.Cu at (129.1, 120.4)
- added Q14: PSMN2R2-40YSD, footprints:LFPAK56, F.Cu at (149.8, 96.6)
- added Q15: DNP, footprints:LFPAK56, F.Cu at (138.2, 112.2)
- added Q16: DNP, footprints:LFPAK56, F.Cu at (138.2, 106.1)
- added Q2: HYG025N06LS1C2, footprints:PDFN_5X6MC_MCH, F.Cu at (141.8, 93.3)
- added Q3: HYG025N06LS1C2, footprints:PDFN_5X6MC_MCH, F.Cu at (133.2, 93.3)
- added Q4: HYG025N06LS1C2, footprints:PDFN_5X6MC_MCH, F.Cu at (152.7, 90.3)
- added Q5: PSMN2R2-40YSD, footprints:LFPAK56, F.Cu at (168.5, 91.4)
- added Q6: PSMN2R2-40YSD, footprints:LFPAK56, F.Cu at (157.6, 97.5)
- added Q7: DNP, footprints:LFPAK56, F.Cu at (146.0, 112.2)
- added Q8: DNP, footprints:LFPAK56, F.Cu at (168.7, 83.5)
- added Q9: PSMN2R2-40YSD, footprints:LFPAK56, F.Cu at (137.1, 118.3)
- added R10: R_2M, footprints:R_0805_OEM, F.Cu at (172.5, 113.1)
- added R11: R_120K, footprints:R_0805_OEM, F.Cu at (195.9, 90.5)
- added R13: DNP, footprints:R_0805_OEM, F.Cu at (113.3, 250.4)
- added R14: R_0, footprints:R_0805_OEM, F.Cu at (117.7, 250.4)
- added R15: DNP, footprints:R_0805_OEM, F.Cu at (113.3, 253.7)
- added R16: R_10K, footprints:R_0805_OEM, F.Cu at (142.6, 227.3)
- added R17: R_0, footprints:R_0805_OEM, F.Cu at (113.3, 257.0)
- added R18: R_10K, footprints:R_0805_OEM, F.Cu at (154.2, 227.3)
- added R19: DNP, footprints:R_0805_OEM, F.Cu at (122.4, 250.4)
- added R2: R_100K, footprints:R_0805_OEM, F.Cu at (176.2, 118.9)
- added R20: R_0, footprints:R_0805_OEM, F.Cu at (122.5, 253.7)
- added R21: R_10K, footprints:R_0805_OEM, F.Cu at (165.9, 227.3)
- added R22: R_1, footprints:R_0805_OEM, F.Cu at (184.9, 111.2)
- added R23: R_1, footprints:R_0805_OEM, F.Cu at (180.8, 114.1)
- added R25: DNP, footprints:R_0805_OEM, F.Cu at (162.1, 127.3)
- added R26: DNP, footprints:R_0805_OEM, F.Cu at (176.6, 113.2)
- added R27: R_0, footprints:R_0805_OEM, F.Cu at (167.5, 121.6)
- added R28: R_1, footprints:R_0805_OEM, F.Cu at (192.6, 96.6)
- added R29: R_1, footprints:R_0805_OEM, F.Cu at (186.4, 102.6)
- added R3: R_1.54K, footprints:R_0805_OEM, F.Cu at (190.6, 105.2)
- added R31: DNP, footprints:R_0805_OEM, F.Cu at (172.1, 116.0)
- added R32: DNP, footprints:R_0805_OEM, F.Cu at (176.6, 110.3)
- added R33: R_0, footprints:R_0805_OEM, F.Cu at (162.5, 124.4)
- added R34: R_1, footprints:R_0805_OEM, F.Cu at (188.4, 99.5)
- added R35: R_1, footprints:R_0805_OEM, F.Cu at (171.6, 121.7)
- added R37: R_0, footprints:R_0805_OEM, F.Cu at (186.4, 105.5)
- added R38: DNP, footprints:R_0805_OEM, F.Cu at (172.1, 118.9)
- added R39: DNP, footprints:R_0805_OEM, F.Cu at (182.3, 105.5)
- added R4: R_845K, footprints:R_0805_OEM, F.Cu at (186.0, 108.3)
- added R40: R_10K, footprints:R_0805_OEM, F.Cu at (166.6, 124.5)
- added R41: R_10K, footprints:R_0805_OEM, F.Cu at (190.6, 102.4)
- added R42: R_10K, footprints:R_0805_OEM, F.Cu at (180.8, 111.2)
- added R43: R_10K, footprints:R_0805_OEM, F.Cu at (176.2, 116.0)
- added R5: R_2M, footprints:R_0805_OEM, F.Cu at (182.3, 102.6)
- added R6: R_300K, footprints:R_0805_OEM, F.Cu at (190.1, 93.7)
- added R7: R_97.6K, footprints:R_0805_OEM, F.Cu at (195.9, 87.6)
- added R8: R_22K, footprints:R_0805_OEM, F.Cu at (157.9, 125.7)
- added R9: R_100K, footprints:R_0805_OEM, F.Cu at (167.9, 115.9)
- added TP1: Test_Point_SMD, footprints:Test_Point_SMD, F.Cu at (142.0, 210.8)
- added TP2: Test_Point_SMD, footprints:Test_Point_SMD, F.Cu at (142.0, 218.4)
- added TP3: Test_Point_SMD, footprints:Test_Point_SMD, F.Cu at (153.7, 210.8)
- added TP4: Test_Point_SMD, footprints:Test_Point_SMD, F.Cu at (153.7, 218.4)
- added TP5: Test_Point_SMD, footprints:Test_Point_SMD, F.Cu at (165.4, 210.8)
- added TP6: Test_Point_SMD, footprints:Test_Point_SMD, F.Cu at (165.4, 218.4)
- added U10: INA240A1D, Package_SO:SOIC-8_3.9x4.9mm_P1.27mm, F.Cu at (130.1, 106.3)
- added U11: INA240A1D, Package_SO:SOIC-8_3.9x4.9mm_P1.27mm, F.Cu at (138.5, 99.8)
- added U12: DRV8320S, footprints:QFN50P500X500X80-33N, F.Cu at (121.4, 122.5)
- added U13: INA240A1D, Package_SO:SOIC-8_3.9x4.9mm_P1.27mm, F.Cu at (130.1, 99.8)
- added U4: TLS4120D0EPVXUMA1, footprints:TLS4120D0EPVXUMA1, F.Cu at (152.3, 83.7)
- added U5: R_500, footprints:R_0805_OEM, F.Cu at (195.9, 84.7)
- added U7: LTC4368CMS-1-PBF, footprints:LTC4368CMS-2-PBF, F.Cu at (174.5, 100.9)
- added U8: LMP8481ASQDGKRQ1, footprints:LMP8481ASQDGKRQ1, F.Cu at (106.2, 216.9)
- added U9: LMP8481ASQDGKRQ1, footprints:LMP8481ASQDGKRQ1, F.Cu at (122.7, 216.9)
Routing:
- net GND: track 65.5 -> 25.5 mm, vias 11 -> 0
- net VCC: track 22.7 -> 0.00 mm
- net Net-(C101-Pad1): track 18.1 -> 0.00 mm
- net Net-(COUT101-Pad1): track 17.3 -> 0.00 mm
- net /12V: track 12.9 -> 0.00 mm
- net Net-(C103-Pad2): track 5.44 -> 0.00 mm
- net Net-(R102-Pad1): track 4.18 -> 0.00 mm
- net Net-(C103-Pad1): track 2.39 -> 0.00 mm
- net Net-(D103-Pad2): track 1.75 -> 0.00 mm
- net Net-(D102-Pad2): track 1.75 -> 0.00 mm
- removed copper zone on F.Cu, net GND
- removed copper zone on F.Cu, net Net-(C103-Pad1)
- removed copper zone on F.Cu, net Net-(C103-Pad2)
- removed copper zone on F.Cu, net Net-(COUT101-Pad1)
Other:
- outline, holes or cut-outs redrawn
- board text removed: "12V"
- board text removed: "5V"
- board text removed: "GND"

Commit message: Laying it out
Parts:
- added R1: R_1m_3W_1%, formula:WSL27261L000FEB, F.Cu at (273.1, 26.7)
- added R12: R_1m_3W_1%, formula:WSL27261L000FEB, F.Cu at (320.0, 26.7)
- added R24: R_1m_3W_1%, formula:WSL27261L000FEB, F.Cu at (382.8, 77.2)
- added R30: R_1m_3W_1%, formula:WSL27261L000FEB, F.Cu at (382.8, 55.0)
- added R36: R_1m_3W_1%, formula:WSL27261L000FEB, F.Cu at (383.0, 34.0)
- added U1: redcube-7461057, formula:redcube_pressfit_6pin, F.Cu at (292.7, -33.7)
- added U2: redcube-7461057, formula:redcube_pressfit_6pin, F.Cu at (292.7, -24.9)
- added U3: redcube-7461057, formula:redcube_pressfit_6pin, F.Cu at (301.5, -33.7)
- added U6: redcube-7461057, formula:redcube_pressfit_6pin, F.Cu at (301.5, -24.9)
- J2, J3: footprint Connector_PinSocket_2.54mm:PinSocket_2x19_P2.54mm_Vertical_SMD -> Connector_PinSocket_2.54mm:PinSocket_2x19_P2.54mm_Vertical
- moved U13 259.0 mm to (383.0, 43.8)
- moved Q16 256.9 mm to (373.6, 208.9)
- moved C58 253.7 mm to (393.7, 40.0)
- moved U10 253.6 mm to (383.0, 87.0)
- moved C52 253.3 mm to (393.4, 60.3)
- moved Q15 251.5 mm to (373.6, 200.7)
- moved Q13 247.7 mm to (363.4, 200.7)
- moved C49 247.4 mm to (388.6, 182.9)
- moved U11 246.9 mm to (383.0, 64.8)
- moved C9 246.3 mm to (320.7, 10.8)
- moved C59 241.9 mm to (388.2, 201.3)
- moved Q14 241.3 mm to (363.4, 208.9)
- moved C54 240.1 mm to (393.7, 44.5)
- moved C57 239.8 mm to (383.2, 212.1)
- moved C47 239.1 mm to (382.6, 193.0)
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
Commit message: buck layout set
Parts:
- added TP11: Test_Point_SMD, TestPoint:TestPoint_Pad_D1.5mm, F.Cu at (141.8, 170.9)
- added TP12: Test_Point_SMD, TestPoint:TestPoint_Pad_D1.5mm, F.Cu at (266.4, -4.70)
- added TP15: Test_Point_SMD, TestPoint:TestPoint_Pad_D1.5mm, F.Cu at (251.4, -4.95)
- added TP16: Test_Point_SMD, TestPoint:TestPoint_Pad_D1.5mm, F.Cu at (248.2, -12.1)
- added TP17: Test_Point_SMD, TestPoint:TestPoint_Pad_D1.5mm, F.Cu at (145.4, 170.9)
- added TP18: Test_Point_SMD, TestPoint:TestPoint_Pad_D1.5mm, F.Cu at (148.9, 167.3)
- added TP20: Test_Point_SMD, TestPoint:TestPoint_Pad_D1.5mm, F.Cu at (145.4, 174.4)
- added TP21: Test_Point_SMD, TestPoint:TestPoint_Pad_D1.5mm, F.Cu at (148.9, 170.9)
- added TP22: Test_Point_SMD, TestPoint:TestPoint_Pad_D1.5mm, F.Cu at (152.5, 167.3)
- added TP23: Test_Point_SMD, TestPoint:TestPoint_Pad_D1.5mm, F.Cu at (152.5, 170.9)
- added TP24: Test_Point_SMD, TestPoint:TestPoint_Pad_D1.5mm, F.Cu at (141.8, 167.3)
- added TP25: Test_Point_SMD, TestPoint:TestPoint_Pad_D1.5mm, F.Cu at (156.0, 167.3)
- added TP26: Test_Point_SMD, TestPoint:TestPoint_Pad_D1.5mm, F.Cu at (152.5, 174.4)
- added TP27: Test_Point_SMD, TestPoint:TestPoint_Pad_D1.5mm, F.Cu at (156.0, 170.9)
- added TP28: Test_Point_SMD, TestPoint:TestPoint_Pad_D1.5mm, F.Cu at (159.6, 167.3)
- added TP29: Test_Point_SMD, TestPoint:TestPoint_Pad_D1.5mm, F.Cu at (156.0, 174.4)
- added TP30: Test_Point_SMD, TestPoint:TestPoint_Pad_D1.5mm, F.Cu at (159.6, 170.9)
- added TP31: Test_Point_SMD, TestPoint:TestPoint_Pad_D1.5mm, F.Cu at (163.1, 167.3)
- added TP32: Test_Point_SMD, TestPoint:TestPoint_Pad_D1.5mm, F.Cu at (159.6, 174.4)
- added TP9: Test_Point_SMD, TestPoint:TestPoint_Pad_D1.5mm, F.Cu at (148.9, 174.4)
- moved J1 308.4 mm to (263.5, -9.08), turned to 270 degrees
- moved R17 297.5 mm to (254.7, -4.70)
- moved C31 293.7 mm to (248.1, -8.45), turned to 180 degrees
- moved R20 292.8 mm to (258.9, -5.40), turned to 90 degrees
- moved C21 292.8 mm to (248.0, -5.21), turned to 180 degrees
- moved R13 292.4 mm to (262.3, -1.15), turned to 270 degrees
- moved R14 292.2 mm to (266.5, -0.95), turned to 180 degrees
- moved R15 291.9 mm to (255.5, -1.27), turned to 270 degrees
- moved C11 286.9 mm to (248.0, -1.91), turned to 180 degrees
- moved R19 286.3 mm to (259.0, -1.21), turned to 270 degrees
- moved U2 202.8 mm to (109.2, 61.3)
- moved C33 192.0 mm to (1.91, 123.8), turned to 90 degrees
- moved TP6 191.5 mm to (1.91, 118.7), turned to 90 degrees
- moved R21 191.2 mm to (5.14, 123.8), turned to 90 degrees
- moved TP5 189.5 mm to (3.43, 112.4)
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Connections:
- C1 pad 1: VBUS -> VS
- C2 pad 1: VBUS -> VS
- C6 pad 1: +10V -> Net-(C6-Pad1)
- C7 pad 1: +10V -> Net-(C6-Pad1)
- J5 pad 1: /INHA -> Net-(J5-Pad1)
- J5 pad 2: Net-(J5-Pad2) -> /INHA
- J6 pad 1: Net-(J5-Pad2) -> Net-(J5-Pad1)
- L1 pad 2: +10V -> Net-(C6-Pad1)
- R10 pad 1: +10V -> Net-(C6-Pad1)
- U4 pad 5: VBUS -> VS
- U4 pad 6: VBUS -> VS
- U4 pad 7: VBUS -> VS

Commit message: additional merge fixes
Parts:
- moved C53 3.56 mm to (343.2, 101.5), turned to 270 degrees
- moved C55 0.57 mm to (337.8, 97.1)

Commit message: more layout, ay
Parts:
- added C61: C_10uF_50V, formula:C_0805_OEM, F.Cu at (326.8, 96.2)
- added C62: C_100nF, formula:C_0603_1608Metric, F.Cu at (328.5, 96.4)
- added H1: MotorConnector_Pad, TestPoint:TestPoint_Pad_4.0x4.0mm, F.Cu at (147.1, 145.9)
- added H2: MotorConnector_Pad, TestPoint:TestPoint_Pad_4.0x4.0mm, F.Cu at (153.1, 145.9)
- added H3: MotorConnector_Pad, TestPoint:TestPoint_Pad_4.0x4.0mm, F.Cu at (159.2, 145.9)
- moved C43 113.7 mm to (297.8, 99.8), turned to 90 degrees
- moved C41 112.4 mm to (295.5, 99.8), turned to 90 degrees
- moved R35 98.8 mm to (356.4, 112.0), turned to 270 degrees
- moved R12 98.0 mm to (227.4, 58.7)
- moved R34 91.4 mm to (364.7, 111.7), turned to 270 degrees
- moved C9 89.2 mm to (245.6, 58.9)
- moved C40 89.0 mm to (303.4, 133.3), turned to 180 degrees
- moved R29 87.8 mm to (335.2, 107.1), turned to 270 degrees
- moved C39 86.9 mm to (303.8, 127.7), turned to 270 degrees
- moved Q15 84.4 mm to (353.3, 118.7), turned to 90 degrees
- moved R24 84.3 mm to (316.5, 129.2), turned to 180 degrees
- moved R26 83.9 mm to (307.0, 133.3)
- moved Q12 82.3 mm to (331.7, 119.6), turned to 270 degrees
- moved R25 82.1 mm to (307.6, 128.1), turned to 270 degrees
- moved Q14 81.3 mm to (377.4, 128.8), turned to 270 degrees
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Connections:
- net Net-(J2-Pad3) renamed /PC12_LED
- net Net-(J2-Pad37) renamed /PC3_LED
- C55 pad 1: GND -> Net-(C55-Pad1)
- U12 pad 23: GND -> Net-(NT2-Pad1)
- U12 pad 31: GND -> Net-(C55-Pad1)

Commit message: layout pushing
Parts:
- moved Q3 2.29 mm to (200.3, 48.8)
- moved R51 0.26 mm to (203.7, 66.0)
- renumbered U5 to R51

Commit message: schem changes, layout changes
Parts:
- added D1: D_TVS_35V, footprints:DO-214AB, F.Cu at (289.3, 2.79)
- added D10: LED_0805, footprints:LED_0805_OEM, F.Cu at (285.6, 31.5)
- added D2: D_TVS_35V, footprints:DO-214AB, F.Cu at (289.3, 13.7)
- added D3: D_TVS_35V, footprints:DO-214AB, F.Cu at (289.3, 21.5)
- added D4: D_TVS_35V, footprints:DO-214AB, F.Cu at (300.9, 13.7)
- added D5: D_TVS_35V, footprints:DO-214AB, F.Cu at (300.9, 21.5)
- added D6: LED_0805, footprints:LED_0805_OEM, F.Cu at (305.4, 30.7)
- added D7: LED_0805, footprints:LED_0805_OEM, F.Cu at (300.4, 31.5)
- added D8: LED_0805, footprints:LED_0805_OEM, F.Cu at (295.5, 31.5)
- added D9: LED_0805, footprints:LED_0805_OEM, F.Cu at (290.5, 31.5)
- added R44: R_0_2512, footprints:R_2512_OEM, F.Cu at (273.6, 32.5)
- added R45: R_0_2512, footprints:R_2512_OEM, F.Cu at (273.6, 25.9)
- added R46: R_430, footprints:R_0805_OEM, F.Cu at (313.8, 25.9)
- added R47: R_68, footprints:R_0805_OEM, F.Cu at (319.3, 19.3)
- added R48: R_160, footprints:R_0805_OEM, F.Cu at (313.8, 23.0)
- added R49: R_68, footprints:R_0805_OEM, F.Cu at (308.2, 27.0)
- added R50: R_68, footprints:R_0805_OEM, F.Cu at (309.9, 29.9)
- added TP10: Test_Point_SMD, footprints:Test_Point_SMD, F.Cu at (309.0, 23.6)
- added TP13: Test_Point_SMD, footprints:Test_Point_SMD, F.Cu at (314.5, 19.6)
- added TP14: Test_Point_SMD, footprints:Test_Point_SMD, F.Cu at (320.5, 15.8)
- added TP19: Test_Point_SMD, footprints:Test_Point_SMD, F.Cu at (309.0, 19.6)
- added TP7: Test_Point_SMD, footprints:Test_Point_SMD, F.Cu at (320.5, 11.8)
- added TP8: Test_Point_SMD, footprints:Test_Point_SMD, F.Cu at (303.4, 27.4)
- C61: footprint formula:C_0805_OEM -> footprints:C_0805_OEM
- C62: footprint formula:C_0603_1608Metric -> footprints:C_0805_OEM
- C9: footprint footprints:C_100uF+ -> footprints:C_0805_OEM
- J2, J3: moved to B.Cu
- R1: footprint formula:WSL27261L000FEB -> footprints:WSL27261L000FEB
- U1, U2, U3, U6: footprint formula:redcube_pressfit_6pin -> footprints:redcube_pressfit_6pin
- moved TP17 165.9 mm to (310.2, 189.7)
- moved TP20 165.9 mm to (310.2, 193.2)
- moved TP31 165.9 mm to (328.0, 186.1)
- moved TP11 165.9 mm to (306.7, 189.7)
- moved TP24 165.9 mm to (306.7, 186.1)
- moved TP25 165.9 mm to (320.9, 186.1)
- moved TP27 165.9 mm to (320.9, 189.7)
- moved TP28 165.9 mm to (324.4, 186.1)
- moved TP29 165.9 mm to (320.9, 193.2)
- moved TP30 165.9 mm to (324.4, 189.7)
- moved TP32 165.9 mm to (324.4, 193.2)
- moved TP18 165.9 mm to (313.8, 186.1)
- moved TP21 165.9 mm to (313.8, 189.7)
- moved TP22 165.9 mm to (317.3, 186.1)
- moved TP23 165.9 mm to (317.3, 189.7)
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Routing:
- net GND: track 25.5 -> 0.00 mm
- added copper zone on F.Cu, net GND
Other:
- board size 109.3 x 58.3 mm -> 109.5 x 121.7 mm
- copper layers 2 -> 4

Commit message: still finishing inverter and other layouts
Parts:
- added NT1: Net-Tie_2, NetTie:NetTie-2_SMD_Pad0.5mm, F.Cu at (217.3, 50.4)
- moved C31 250.6 mm to (31.3, 117.3)
- moved C11 250.6 mm to (31.3, 123.9)
- moved C21 250.6 mm to (31.3, 120.6)
- moved J1 250.6 mm to (46.7, 116.7)
- moved R13 250.6 mm to (45.5, 124.6)
- moved R14 250.6 mm to (49.7, 124.8)
- moved R15 250.6 mm to (38.7, 124.5)
- moved R17 250.6 mm to (37.9, 121.1)
- moved R19 250.6 mm to (42.2, 124.6)
- moved R20 250.6 mm to (42.1, 120.4)
- moved TP12 250.6 mm to (49.6, 121.1)
- moved TP15 250.6 mm to (34.6, 120.8)
- moved TP16 250.6 mm to (31.4, 113.7)
- moved R45 208.9 mm to (95.8, 135.5), turned to 90 degrees
- moved R44 206.2 mm to (101.3, 145.9), turned to 270 degrees
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Connections:
- R12 pad 1: Net-(Q3-Pad1) -> VBUS
- R12 pad 2: /SYSTEM_SH_+ -> /SYSTEM_SH_-
- R12 pad 3: /SYSTEM_SH_- -> /SYSTEM_SH_+
- R12 pad 4: VBUS -> Net-(Q3-Pad1)
Routing:
- removed copper zone on B.Cu, net GND
- removed copper zone on F.Cu, net GND
Other:
- board size 109.5 x 121.7 mm -> 118 x 121.9 mm
