File: bldc_foc_controller/bldc_foc_controller.kicad_pcb (KiCad board)
At the start: 4 copper layers, 118 x 121.9 mm, 196 parts, among them J1 Conn_01x05, J2 Conn_02x19_Odd_Even, J3 Conn_02x19_Odd_Even, J4 Conn_01x10, J5 CONN_01x02, J6 CONN_01X03, J7 CONN_01x02, J8 CONN_01x02, Q1 HYG025N06LS1C2, Q10 PSMN2R2-40YSD, Q11 DNP, Q12 DNP, Q13 PSMN2R2-40YSD, Q14 PSMN2R2-40YSD, Q15 DNP, Q16 DNP, Q2 HYG025N06LS1C2, Q3 HYG025N06LS1C2, Q4 HYG025N06LS1C2, Q5 PSMN2R2-40YSD, Q6 PSMN2R2-40YSD, Q7 DNP, Q8 DNP, Q9 PSMN2R2-40YSD, U1 redcube-7461057, U10 INA240A1D, U11 INA240A1D, U12 DRV8320S, U13 INA240A1D, U2 redcube-7461057, U3 redcube-7461057, U4 TLS4120D0EPVXUMA1, U6 redcube-7461057, U7 LTC4368CMS-1-PBF, U8 LMP8481ASQDGKRQ1, U9 LMP8481ASQDGKRQ1

Commit message: moving comps to the board
Parts:
- added NT2: Net-Tie_2, NetTie:NetTie-2_SMD_Pad0.5mm, F.Cu at (138.2, 89.5)
- R36: footprint formula:WSL27261L000FEB -> footprints:WSL27261L000FEB
- moved C59 300.8 mm to (101.5, 67.8), turned to 90 degrees
- moved R38 300.3 mm to (103.7, 67.0)
- moved C58 299.1 mm to (95.0, 55.1), turned to 180 degrees
- moved C60 297.6 mm to (99.1, 67.8), turned to 90 degrees
- moved C56 297.1 mm to (103.7, 63.4), turned to 90 degrees
- moved R37 295.2 mm to (98.6, 55.1)
- moved C54 291.7 mm to (102.3, 58.0), turned to 270 degrees
- moved R39 289.0 mm to (107.2, 63.4), turned to 90 degrees
- moved C57 283.8 mm to (107.2, 66.9)
- moved U13 280.1 mm to (103.0, 52.3), turned to 270 degrees
- moved R36 267.5 mm to (115.2, 52.4), turned to 90 degrees
- moved TP19 266.2 mm to (46.5, 64.0)
- moved Q16 265.4 mm to (111.6, 62.2), turned to 90 degrees
- moved C48 265.3 mm to (128.4, 53.3), turned to 270 degrees
- moved TP26 261.6 mm to (96.9, 52.3), turned to 180 degrees
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Connections:
- C53 pad 2: GND -> Net-(C53-Pad2)
- R30 pad 1: /PH_B -> /PH_B_SH
- R30 pad 4: /PH_B_SH -> /PH_B
- R36 pad 1: /PH_C -> /PH_C_SH
- R36 pad 4: /PH_C_SH -> /PH_C
- U11 pad 1: Net-(R30-Pad2) -> Net-(R30-Pad3)
- U11 pad 8: Net-(R30-Pad3) -> Net-(R30-Pad2)
- U12 pad 23: Net-(NT2-Pad1) -> Net-(C53-Pad1)
- U12 pad 24: Net-(C53-Pad1) -> Net-(C53-Pad2)
- U13 pad 1: Net-(R36-Pad2) -> Net-(R36-Pad3)
- U13 pad 8: Net-(R36-Pad3) -> Net-(R36-Pad2)

Commit message: housekeeping
Parts:
- moved D8 278.0 mm to (17.2, 227.8)
- moved D9 278.0 mm to (17.2, 230.0)
- moved NT1 278.0 mm to (17.8, 244.0)
- moved R46 278.0 mm to (21.3, 234.1)
- moved R48 278.0 mm to (21.3, 232.1)
- moved R49 278.0 mm to (21.3, 230.0)
- moved R50 278.0 mm to (21.3, 236.2)
- moved D10 278.0 mm to (17.2, 236.2)
- moved D6 278.0 mm to (17.2, 232.1)
- moved D7 278.0 mm to (17.2, 234.1)
- moved R47 278.0 mm to (21.3, 227.8)
- moved TP22 260.4 mm to (133.9, 301.3), turned to 90 degrees
- moved C44 256.3 mm to (133.8, 297.9), turned to 90 degrees
- moved R27 255.3 mm to (131.0, 298.9), turned to 180 degrees
- moved H3 253.5 mm to (146.4, 286.4), turned to 90 degrees
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Other:
- board text added: "deadspace"

Commit message: major layout update
Parts:
- moved J4 103.7 mm to (190.6, 175.5)
- moved J6 103.7 mm to (203.8, 184.7)
- moved R14 103.7 mm to (169.0, 180.2)
- moved R16 103.7 mm to (173.2, 205.0)
- moved R17 103.7 mm to (172.8, 168.4)
- moved TP12 103.7 mm to (172.8, 180.0)
- moved C11 103.7 mm to (170.0, 161.7)
- moved C16 103.7 mm to (170.0, 205.0)
- moved C30 103.7 mm to (176.5, 205.0)
- moved C31 103.7 mm to (176.5, 161.7)
- moved C33 103.7 mm to (182.9, 204.9)
- moved J1 103.7 mm to (177.2, 177.1)
- moved J7 103.7 mm to (209.7, 185.2)
- moved J8 103.7 mm to (209.7, 180.4)
- moved R13 103.7 mm to (169.2, 175.9)
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Routing:
- net /VBUS_UNPROTECTED: track 0.00 -> 69.2 mm
- net Net-(Q1-Pad2): track 0.00 -> 48.8 mm
- net GND: track 0.00 -> 45.2 mm
- net /PH_A_SH: track 0.00 -> 41.1 mm
- net Net-(Q3-Pad1): track 0.00 -> 35.2 mm
- net /GHA: track 0.00 -> 32.2 mm
- net /GLA: track 0.00 -> 30.3 mm
- net /PH_C_SH: track 0.00 -> 27.6 mm
- net VBUS: track 0.00 -> 23.9 mm
- net Net-(C6-Pad1): track 0.00 -> 22.3 mm
- net /PH_B_SH: track 0.00 -> 20.5 mm
- net /GLB: track 0.00 -> 17.2 mm
- net Net-(R30-Pad3): track 0.00 -> 15.3 mm
- net Net-(R30-Pad2): track 0.00 -> 14.9 mm
- net /GLC: track 0.00 -> 14.7 mm
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- added copper zone on F.Cu, net GND
- added copper zone on F.Cu, net Net-(L1-Pad1)
- added copper zone on F.Cu, net VBUS
Other:
- board text removed: "deadspace"

Commit message: quick layout push
Parts:
- moved R11 5.65 mm to (82.2, 255.0)
- moved C2 5.65 mm to (80.6, 239.6)
- moved C6 5.65 mm to (81.3, 258.3)
- moved C7 5.65 mm to (79.3, 258.9)
- moved C9 5.65 mm to (81.6, 267.2)
- moved D7 5.65 mm to (85.6, 240.9)
- moved R44 5.65 mm to (86.4, 247.1)
- moved R46 5.65 mm to (84.7, 237.8)
- moved R9 5.65 mm to (82.2, 252.6)
- moved U4 5.65 mm to (81.3, 247.2)
- moved D5 5.65 mm to (75.5, 265.7)
- moved L1 5.65 mm to (77.6, 253.8)
- moved R10 5.65 mm to (83.4, 258.3)
- moved R45 5.65 mm to (75.3, 246.7)
- moved TP10 5.65 mm to (75.9, 258.8)
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Routing:
- net /VBUS_UNPROTECTED: track 69.2 -> 34.5 mm
- net Net-(Q3-Pad1): track 35.2 -> 37.9 mm

Commit message: quick layout push
Parts:
- moved C41 142.9 mm to (123.2, 160.0)
- moved Q2 142.9 mm to (69.7, 163.3)
- moved U3 142.9 mm to (110.4, 177.9)
- moved C1 142.9 mm to (75.0, 98.9)
- moved C10 142.9 mm to (119.6, 167.0)
- moved C11 142.9 mm to (164.6, 18.9)
- moved C12 142.9 mm to (107.6, 144.1)
- moved C13 142.9 mm to (110.1, 144.1)
- moved C14 142.9 mm to (112.6, 144.1)
- moved C15 142.9 mm to (115.1, 144.1)
- moved C17 142.9 mm to (105.1, 148.9)
- moved C18 142.9 mm to (102.6, 148.9)
- moved C19 142.9 mm to (100.1, 148.9)
- moved C2 142.9 mm to (75.2, 96.7)
- moved C20 142.9 mm to (97.6, 148.9)
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Other:
- board outline removed

Commit message: added manufacturing
Parts:
- moved C9 7.99 mm to (84.3, 124.8)
- moved D5 7.99 mm to (78.1, 123.3)
- moved D1 1.58 mm to (79.6, 164.1)
Routing:
- net Net-(Q3-Pad1): track 37.9 -> 0.61 mm
- net /VBUS_UNPROTECTED: track 34.5 -> 17.8 mm
- net VBUS: track 23.9 -> 25.7 mm
- added copper zone on F.Cu, net /VBUS_UNPROTECTED
- added copper zone on F.Cu, net Net-(Q3-Pad1)
Changed lines of the file:
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@@
     (thickness 1.6)
     (drawings 15)
-    (tracks 398)
+    (tracks 380)
     (zones 0)
     (modules 197)
@@
     (trace_clearance 0.1524)
     (zone_clearance 0.1524)
-    (zone_45_only no)
+    (zone_45_only yes)
     (trace_min 0.1524)
     (via_size 0.6096)
@@
   )
   (module footprints:DO-214AB (layer F.Cu)
-    (at 70.1421 122.8471)
+    (at 78.1177 123.3043)
     (fp_text reference D5 (at 0.508 -0.3175) (layer F.SilkS)
       (effects (font (size 1 1) (thickness 0.15)))
@@
   )
   (module footprints:DO-214AB (layer F.Cu)
-    (at 79.0575 162.5854)
-    (fp_text reference D1 (at -1.905 -4.445) (layer F.SilkS)
+    (at 79.5528 164.084)
+    (fp_text reference D1 (at 2.794 -4.064) (layer F.SilkS)
       (effects (font (size 1 1) (thickness 0.15)))
     )
@@
   )
   (module footprints:C_0805_OEM (layer F.Cu)
-    (at 76.3016 124.3711 90)
+    (at 84.2772 124.8283 90)
     (descr "Capacitor SMD 0805, reflow soldering, AVX (see smccp.pdf)")
     (tags "capacitor 0805")
@@
   (segment (start 78.3996 96.6216) (end 78.2066 96.8146) (width 0.5) (layer F.Cu) (net 1))
   (segment (start 78.3996 94.9706) (end 78.3996 96.6216) (width 0.5) (layer F.Cu) (net 1))
-  (segment (start 75.7776 122.8471) (end 76.3016 123.3711) (width 0.5) (layer F.Cu) (net 1))
-  (segment (start 73.6271 122.8471) (end 75.7776 122.8471) (width 0.5) (layer F.Cu) (net 1))
+  (segment (start 83.7532 123.3043) (end 84.2772 123.8283) (width 0.5) (layer F.Cu) (net 1))
+  (segment (start 81.6027 123.3043) (end 83.7532 123.3043) (width 0.5) (layer F.Cu) (net 1))
   (segment (start 87.945 156.0424) (end 87.945 156.6164) (width 0.254) (layer F.Cu) (net 1))
   (segment (start 87.4395 155.5369) (end 87.945 156.0424) (width 0.254) (layer F.Cu) (net 1))
@@
   (segment (start 78.9305 144.1544) (end 78.9305 145.6309) (width 0.381) (layer F.Cu) (net 1))
   (segment (start 106.226893 119.858507) (end 107.615286 121.2469) (width 0.1524) (layer F.Cu) (net 2))
-  (segment (start 75.8952 127.6604) (end 73.8632 129.6924) (width 0.5) (layer F.Cu) (net 2))
-  (segment (start 75.8952 126.9967) (end 75.8952 127.6604) (width 0.5) (layer F.Cu) (net 2))
   (segment (start 106.163393 119.875721) (end 107.869286 121.581614) (width 0.381) (layer F.Cu) (net 2))
   (segment (start 106.163393 119.731507) (end 106.163393 119.875721) (width 0.381) (layer F.Cu) (net 2))
@@
   (segment (start 140.8557 110.8442) (end 142.645 109.0549) (width 0.381) (layer F.Cu) (net 2))
   (segment (start 140.8557 111.4298) (end 140.8557 110.8442) (width 0.381) (layer F.Cu) (net 2))
+  (segment (start 76.3016 127.254) (end 75.2602 128.2954) (width 0.5) (layer F.Cu) (net 2))
+  (segment (start 84.2772 125.8283) (end 84.2772 127.7112) (width 0.5) (layer F.Cu) (net 2))
+  (segment (start 75.2602 128.2954) (end 73.8632 129.6924) (width 0.5) (layer F.Cu) (net 2))
   (segment (start 80.74 147.6339) (end 80.4545 147.9194) (width 0.381) (layer F.Cu) (net 3))
   (segment (start 80.5495 146.2024) (end 80.5495 147.6339) (width 0.381) (layer F.Cu) (net 3))
@@
   (segment (start 82.197699 152.6921) (end 82.295291 152.594508) (width 0.5) (layer F.Cu) (net 4))
   (segment (start 80.518 152.6921) (end 82.197699 152.6921) (width 0.5) (layer F.Cu) (net 4))
-  (segment (start 71.628 166.6494) (end 72.4535 165.8239) (width 0.381) (layer F.Cu) (net 4))
-  (segment (start 64.8335 166.6494) (end 71.628 166.6494) (width 0.381) (layer F.Cu) (net 4))
-  (segment (start 63.119 164.9349) (end 64.8335 166.6494) (width 0.381) (layer F.Cu) (net 4))
-  (segment (start 63.119 157.3149) (end 63.119 164.9349) (width 0.381) (layer F.Cu) (net 4))
-  (segment (start 72.4535 165.8239) (end 72.4535 165.1889) (width 0.381) (layer F.Cu) (net 4))
-  (segment (start 64.135 156.2989) (end 63.119 157.3149) (width 0.381) (layer F.Cu) (net 4))
-  (segment (start 64.5795 156.2989) (end 64.135 156.2989) (width 0.381) (layer F.Cu) (net 4))
-  (segment (start 78.552 159.6059) (end 75.5725 162.5854) (width 0.381) (layer F.Cu) (net 4))
-  (segment (start 78.552 154.9019) (end 78.552 159.6059) (width 0.381) (layer F.Cu) (net 4))
+  (segment (start 72.4535 165.1889) (end 72.4535 162.6489) (width 0.5) (layer F.Cu) (net 4))
+  (segment (start 78.552 161.5998) (end 76.0678 164.084) (width 0.5) (layer F.Cu) (net 4))
+  (segment (start 78.552 154.9019) (end 78.552 161.5998) (width 0.5) (layer F.Cu) (net 4))
   (segment (start 79.033999 142.257899) (end 78.9305 142.1544) (width 0.254) (layer F.Cu) (net 5))
   (segment (start 81.54035 142.257899) (end 79.033999 142.257899) (width 0.254) (layer F.Cu) (net 5))
@@
   (segment (start 73.3552 158.9024) (end 76.7715 155.4861) (width 0.381) (layer F.Cu) (net 44))
   (segment (start 73.4314 134.1882) (end 73.8632 134.62) (width 0.381) (layer F.Cu) (net 46))
-  (segment (start 71.6788 136.8044) (end 73.8632 134.62) (width 0.5) (layer F.Cu) (net 46))
-  (segment (start 65.9765 136.8044) (end 71.6788 136.8044) (width 0.5) (layer F.Cu) (net 46))
-  (segment (start 64.516 138.2649) (end 65.9765 136.8044) (width 0.5) (layer F.Cu) (net 46))
-  (segment (start 64.516 138.5824) (end 64.516 138.2649) (width 0.5) (layer F.Cu) (net 46))
-  (segment (start 64.516 138.5824) (end 64.516 141.1224) (width 0.5) (layer F.Cu) (net 46))
-  (segment (start 72.5805 149.6949) (end 72.5805 147.1549) (width 0.5) (layer F.Cu) (net 46))
-  (segment (start 72.5805 149.6949) (end 72.5805 149.9743) (width 0.5) (layer F.Cu) (net 46))
-  (segment (start 72.5805 149.9743) (end 71.374 151.1808) (width 0.5) (layer F.Cu) (net 46))
-  (segment (start 71.374 151.1808) (end 64.4652 151.1808) (width 0.5) (layer F.Cu) (net 46))
-  (segment (start 64.4652 151.1808) (end 62.738 149.4536) (width 0.5) (layer F.Cu) (net 46))
-  (segment (start 63.5207 141.1224) (end 64.516 141.1224) (width 0.5) (layer F.Cu) (net 46))
-  (segment (start 62.738 141.9051) (end 63.5207 141.1224) (width 0.5) (layer F.Cu) (net 46))
-  (segment (start 62.738 149.4536) (end 62.738 141.9051) (width 0.5) (layer F.Cu) (net 46))
   (segment (start 121.473 142.9639) (end 129.3225 142.9639) (width 0.254) (layer F.Cu) (net 47))
   (segment (start 129.3225 142.9639) (end 130.2065 143.8479) (width 0.254) (layer F.Cu) (net 47))
@@
       )
     )
+  )
+  (zone (net 46) (net_name "Net-(Q3-Pad1)") (layer F.Cu) (hatch edge 0.508)
+    (connect_pads yes (clearance 0.1524))
+    (min_thickness 0.254)
+    (fill yes (arc_segments 32) (thermal_gap 0.508) (thermal_bridge_width 0.508))
+    (polygon
+      (pts
+        (xy 76.6572 137.3124) (xy 66.4464 137.3124) (xy 65.786 137.9728) (xy 65.786 141.6812) (xy 65.786 141.8336)
+        (xy 63.8048 141.8336) (xy 63.6016 142.0368) (xy 63.6016 142.9512) (xy 65.6336 145.034) (xy 65.6336 150.4696)
+        (xy 71.374 150.4696) (xy 71.374 146.3548) (xy 73.0504 146.3548) (xy 74.0156 146.3548) (xy 74.080036 152.8064)
+        (xy 61.034331 152.8064) (xy 60.9092 133.1468) (xy 70.6628 133.1468) (xy 76.6572 133.1468)
+      )
+    )
+  )
+  (zone (net 4) (net_name /VBUS_UNPROTECTED) (layer F.Cu) (hatch edge 0.508)
+    (connect_pads yes (clearance 0.1524))
+    (min_thickness 0.254)
+    (fill yes (arc_segments 32) (thermal_gap 0.508) (thermal_bridge_width 0.508))
+    (polygon
+      (pts
+        (xy 65.2272 156.718) (xy 65.024 156.9212) (xy 63.9064 156.9212) (xy 63.3984 157.4292) (xy 63.3984 162.339506)
+        (xy 65.7352 166.2176) (xy 71.6788 166.2176) (xy 71.6788 162.2552) (xy 74.168 162.2552) (xy 78.0288 158.3944)
+        (xy 78.0288 154.0764) (xy 79.0956 154.0764) (xy 79.0956 160.3756) (xy 80.9752 162.2552) (xy 81.0768 162.2552)
+        (xy 81.0768 181.7116) (xy 59.2836 181.7116) (xy 59.2836 153.3652) (xy 65.2272 153.3652)
+      )
+    )
